Commit message: Rework gripper controllers.

File: boxbot_description/urdf/servos.urdf.xacro (robot description, xacro)
@@ -69,4 +69,14 @@
     </actuator>
   </transmission>
+  <transmission name="ltran_fake">
+    <type>transmission_interface/SimpleTransmission</type>
+    <joint name="left_gripper_prismatic_joint_2">
+      <hardwareInterface>hardware_interface/PositionJointInterface</hardwareInterface>
+    </joint>
+    <actuator name="left_motor_fake">
+      <hardwareInterface>hardware_interface/PositionJointInterface</hardwareInterface>
+      <mechanicalReduction>1</mechanicalReduction>
+    </actuator>
+  </transmission>
   <!--right-->
   <transmission name="rtran1">
@@ -123,5 +133,5 @@
     <type>transmission_interface/SimpleTransmission</type>
     <joint name="right_gripper_joint">
-       <hardwareInterface>hardware_interface/PositionJointInterface</hardwareInterface>
+      <hardwareInterface>hardware_interface/PositionJointInterface</hardwareInterface>
     </joint>
     <actuator name="right_motor6">
@@ -130,3 +140,13 @@
     </actuator>
   </transmission>
+  <transmission name="rtran_fake">
+    <type>transmission_interface/SimpleTransmission</type>
+    <joint name="right_gripper_prismatic_joint_2">
+      <hardwareInterface>hardware_interface/PositionJointInterface</hardwareInterface>
+    </joint>
+    <actuator name="right_motor_fake">
+      <hardwareInterface>hardware_interface/PositionJointInterface</hardwareInterface>
+      <mechanicalReduction>1</mechanicalReduction>
+    </actuator>
+  </transmission>
 </robot>

Commit message: Switch joint controllers to individual position contollers and fix the gazebo joint mimic.

File: boxbot_description/urdf/servos.urdf.xacro (robot description, xacro)
@@ -69,14 +69,4 @@
     </actuator>
   </transmission>
-  <transmission name="ltran_fake">
-    <type>transmission_interface/SimpleTransmission</type>
-    <joint name="left_gripper_prismatic_joint_2">
-      <hardwareInterface>hardware_interface/PositionJointInterface</hardwareInterface>
-    </joint>
-    <actuator name="left_motor_fake">
-      <hardwareInterface>hardware_interface/PositionJointInterface</hardwareInterface>
-      <mechanicalReduction>1</mechanicalReduction>
-    </actuator>
-  </transmission>
   <!--right-->
   <transmission name="rtran1">
@@ -140,13 +130,3 @@
     </actuator>
   </transmission>
-  <transmission name="rtran_fake">
-    <type>transmission_interface/SimpleTransmission</type>
-    <joint name="right_gripper_prismatic_joint_2">
-      <hardwareInterface>hardware_interface/PositionJointInterface</hardwareInterface>
-    </joint>
-    <actuator name="right_motor_fake">
-      <hardwareInterface>hardware_interface/PositionJointInterface</hardwareInterface>
-      <mechanicalReduction>1</mechanicalReduction>
-    </actuator>
-  </transmission>
 </robot>
