Commit message: Update WidowX arm with measured masses.

File: boxbot_description/urdf/widowx.urdf.xacro (robot description, xacro)
@@ -42,5 +42,5 @@
          <inertial>
             <origin xyz="0 0 0" rpy="0 0 0" />
-            <mass value="1" />
+            <mass value="0.061" />
             <inertia ixx="1.0" ixy="0.0" ixz="0.0" iyy="1.0" iyz="0.0" izz="1.0" />
          </inertial>
@@ -62,5 +62,5 @@
          <inertial>
             <origin xyz="0 0 0" rpy="0 0 0" />
-            <mass value="1" />
+            <mass value="3.62e-1" />
             <inertia ixx="1.0" ixy="0.0" ixz="0.0" iyy="1.0" iyz="0.0" izz="1.0" />
          </inertial>
@@ -82,5 +82,5 @@
          <inertial>
             <origin xyz="0 0 0" rpy="0 0 0" />
-            <mass value="1" />
+            <mass value="1.87e-1" />
             <inertia ixx="1.0" ixy="0.0" ixz="0.0" iyy="1.0" iyz="0.0" izz="1.0"/>
          </inertial>
@@ -102,5 +102,5 @@
          <inertial>
             <origin xyz="0 0 0" rpy="0 0 0" />
-            <mass value="1" />
+            <mass value="9.1e-2" />
             <inertia ixx="1.0" ixy="0.0" ixz="0.0" iyy="1.0" iyz="0.0" izz="1.0" />
          </inertial>
@@ -122,5 +122,5 @@
          <inertial>
             <origin xyz="0 0 0" rpy="0 0 0" />
-            <mass value="1" />
+            <mass value="6.3e-2" />
             <inertia ixx="1.0" ixy="0.0" ixz="0.0" iyy="1.0" iyz="0.0" izz="1.0" />
          </inertial>

File: boxbot_description/urdf/widowx_gripper.xacro (robot description, xacro)
@@ -18,5 +18,5 @@
       <inertial>
          <origin xyz="0 0 0" rpy="0 0 0" />
-         <mass value="1" />
+         <mass value="7.0e-3" />
          <inertia ixx="1.0" ixy="0.0" ixz="0.0" iyy="1.0" iyz="0.0" izz="1.0" />
       </inertial>
@@ -40,5 +40,5 @@
       <inertial>
          <origin xyz="0 0 0" rpy="0 0 0" />
-         <mass value="1" />
+         <mass value="8.0e-3" />
          <inertia ixx="1.0" ixy="0.0" ixz="0.0" iyy="1.0" iyz="0.0" izz="1.0" />
       </inertial>
@@ -60,5 +60,5 @@
       <inertial>
          <origin xyz="0 0 0" rpy="0 0 0" />
-         <mass value="1" />
+         <mass value="8.0e-3" />
          <inertia ixx="1.0" ixy="0.0" ixz="0.0" iyy="1.0" iyz="0.0" izz="1.0" />
       </inertial>
