Commit message: Make slight adjustment to test blocks.

File: boxbot_description/urdf/test_block.urdf.xacro (robot description, xacro)
@@ -9,5 +9,5 @@
       </inertial>
       <visual>
-        <origin xyz="0.0 0.0 0.0"/>
+        <origin xyz="0.0 0.0 0.0381"/>
         <geometry>
           <box size="0.0762 0.01905 0.0762"/>
@@ -15,5 +15,5 @@
       </visual>
       <collision>
-        <origin xyz="0.0 0.0 0.0"/>
+        <origin xyz="0.0 0.0 0.0381"/>
         <geometry>
           <box size="0.0762 0.01905 0.0762 "/>
@@ -22,5 +22,5 @@
     </link>
     <joint name="${prefix}test_block_joint" type="fixed">
-      <origin xyz="0.0 0.0 0.0889" />
+      <origin xyz="0.0 0.0 0.0508" />
       <parent link="${parent}" />
       <child link="${prefix}test_block"/>
