Commit message: Add initial collision and inertial properties for new links.

File: boxbot_description/robots/boxbot.urdf (robot description, URDF)
Before this commit: robot boxbot, 21 links, 20 joints
Links:
- link base_link: mass None -> 1
- link torso: mass None -> 1; geometry collision box size=0.20 0.12 0.35; visual box size=0.20 0.12 0.35

File: boxbot_description/robots/boxbot.urdf.xacro (robot description, xacro)
@@ -1,4 +1,5 @@
 <?xml version="1.0"?>
 <robot name="boxbot" xmlns:xacro="http://ros.org/wiki/xacro">
+  <xacro:include filename="$(find widowx_arm_description)/urdf/common_materials.xacro" />
   <link name="world"/>
   <link name="base_link">
@@ -7,5 +8,13 @@
         <box size="0.3048 0.3048 0.00635"/>
       </geometry>
+      <xacro:material_yellow/>
     </visual>
+    <!--Can't get collision to work for this link; likely a collision issue with the torso.-->
+    <inertial>
+      <!--placeholders-->
+      <origin xyz="0.1524 0.1524 0.003175" rpy="0 0 0"/>
+      <mass value="1"/>
+      <inertia ixx="1.0" ixy="0.0" ixz="0.0" iyy="1.0" iyz="0.0" izz="1.0"/>
+    </inertial>
   </link>
   <link name="torso">
@@ -14,5 +23,17 @@
         <box size="0.20 0.12 0.35"/>
       </geometry>
+      <xacro:material_yellow/>
     </visual>
+    <collision>
+      <geometry>
+        <box size="0.20 0.12 0.35"/>
+      </geometry>
+    </collision>
+    <inertial>
+      <!--placeholders-->
+      <origin xyz="0.100 0.060 0.175" rpy="0 0 0"/>
+      <mass value="1"/>
+      <inertia ixx="1.0" ixy="0.0" ixz="0.0" iyy="1.0" iyz="0.0" izz="1.0"/>
+    </inertial>
   </link>
   <joint name="fixed" type="fixed">

Commit message: Added mimicking functionality for the grippers in the Gazebo simulation using the University of Patras Robotics Group's Gazebo mimic joint plugin.

File: boxbot_description/robots/boxbot.urdf (robot description, URDF)
Before this commit: robot boxbot, 21 links, 20 joints
Links:
- link left_gripper_rail_link: geometry visual mesh filename=package://boxbot_description/meshes/gripper_rail_link.stl
- link right_gripper_rail_link: geometry visual mesh filename=package://boxbot_description/meshes/gripper_rail_link.stl

File: boxbot_description/robots/boxbot.urdf.xacro (robot description, xacro)
@@ -55,3 +55,4 @@
   </xacro:widowx_arm>
   <xacro:include filename="$(find boxbot_description)/urdf/servos.urdf.xacro"/>
+  <xacro:include filename="$(find boxbot_description)/urdf/joint_mimic.gazebo"/>
 </robot>

File: boxbot_description/urdf/widowx_gripper.xacro (robot description, xacro)
@@ -9,10 +9,11 @@
          <xacro:material_black />
       </visual>
-      <collision>
+      <!--Removed for now due to problems with collision in Gazebo-->
+      <!--collision>
          <origin xyz="0 0 0" rpy="0 0 1.57" />
          <geometry>
             <mesh filename="package://boxbot_description/meshes/gripper_rail_link.stl"/>
          </geometry>
-      </collision>
+      </collision-->
       <inertial>
          <origin xyz="0 0 0" rpy="0 0 0" />

Commit message: Update Boxbot model to reflect current hardware design; remove gazebo_joint_mimic plugin.

File: boxbot_description/robots/boxbot.urdf (robot description, URDF)
Before this commit: robot boxbot, 21 links, 20 joints
Links:
- link base_link: geometry visual box size=0.3048 0.3048 0.01905
- link left_biceps_link: mass 1 -> 3.62e-1
- link left_forearm_link: mass 1 -> 1.87e-1
- link left_gripper_1_link: mass 1 -> 8.0e-3
- link left_gripper_2_link: mass 1 -> 8.0e-3
- link left_gripper_rail_link: mass 1 -> 7.0e-3
- link left_shoulder_link: mass 1 -> 0.061
- link left_wrist_1_link: mass 1 -> 9.1e-2
- link left_wrist_2_link: mass 1 -> 6.3e-2
- link right_biceps_link: mass 1 -> 3.62e-1
- link right_forearm_link: mass 1 -> 1.87e-1
- link right_gripper_1_link: mass 1 -> 8.0e-3
- link right_gripper_2_link: mass 1 -> 8.0e-3
- link right_gripper_rail_link: mass 1 -> 7.0e-3
- link right_shoulder_link: mass 1 -> 0.061
- link right_wrist_1_link: mass 1 -> 9.1e-2
- link right_wrist_2_link: mass 1 -> 6.3e-2
- link torso: geometry collision box size=0.19685 0.12065 0.3556; visual box size=0.19685 0.12065 0.3556
Joints:
- joint fixed: origin (none) -> xyz=0 0 0.009525 rpy=0 0 0
- joint left_arm_base_joint: origin xyz=0 0.087 0.0877273 rpy=-1.5707963268 0 0 -> xyz=0 0.087325 0.0635 rpy=-1.5707963268 0 0
- joint right_arm_base_joint: origin xyz=0 -0.087 0.0877273 rpy=1.5707963268 0 0 -> xyz=0 -0.087325 0.0635 rpy=1.5707963268 0 0
- joint waist_joint: origin xyz=0 0 0.178175 rpy=0 0 0 -> xyz=0 0 0.187325 rpy=0 0 0

File: boxbot_description/robots/boxbot.urdf.xacro (robot description, xacro)
@@ -6,5 +6,5 @@
     <visual>
       <geometry>
-        <box size="0.3048 0.3048 0.00635"/>
+        <box size="0.3048 0.3048 0.01905"/>
       </geometry>
       <xacro:material_yellow/>
@@ -13,5 +13,5 @@
     <inertial>
       <!--placeholders-->
-      <origin xyz="0.1524 0.1524 0.003175" rpy="0 0 0"/>
+      <origin xyz="0.1524 0.1524 0.009525" rpy="0 0 0"/>
       <mass value="1"/>
       <inertia ixx="1.0" ixy="0.0" ixz="0.0" iyy="1.0" iyz="0.0" izz="1.0"/>
@@ -21,5 +21,5 @@
     <visual>
       <geometry>
-        <box size="0.20 0.12 0.35"/>
+        <box size="0.19685 0.12065 0.3556"/>
       </geometry>
       <xacro:material_yellow/>
@@ -27,10 +27,10 @@
     <collision>
       <geometry>
-        <box size="0.20 0.12 0.35"/>
+        <box size="0.19685 0.12065 0.3556"/>
       </geometry>
     </collision>
     <inertial>
       <!--placeholders-->
-      <origin xyz="0.100 0.060 0.175" rpy="0 0 0"/>
+      <origin xyz="0.098425 0.060325 0.1778" rpy="0 0 0"/>
       <mass value="1"/>
       <inertia ixx="1.0" ixy="0.0" ixz="0.0" iyy="1.0" iyz="0.0" izz="1.0"/>
@@ -38,9 +38,10 @@
   </link>
   <joint name="fixed" type="fixed">
+    <origin xyz="0 0 0.009525" rpy="0 0 0"/>
     <parent link="world"/>
     <child link="base_link"/>
   </joint>
   <joint name="waist_joint" type="fixed">
-    <origin xyz="0 0 0.178175" rpy="0 0 0"/>
+    <origin xyz="0 0 0.187325" rpy="0 0 0"/>
     <parent link="base_link"/>
     <child link="torso"/>
@@ -48,12 +49,11 @@
   <xacro:include filename="$(find boxbot_description)/urdf/widowx.urdf.xacro"/>
   <xacro:widowx_arm parent="torso" prefix="left_">
-    <origin xyz="0 0.087 0.0877273" rpy="-1.5707963268 0 0"/>
+    <origin xyz="0 0.087325 0.0635" rpy="-1.5707963268 0 0"/>
   </xacro:widowx_arm>
   <xacro:include filename="$(find boxbot_description)/urdf/widowx.urdf.xacro"/>
   <xacro:widowx_arm parent="torso" prefix="right_">
-    <origin xyz="0 -0.087 0.0877273" rpy="1.5707963268 0 0"/>
+    <origin xyz="0 -0.087325 0.0635" rpy="1.5707963268 0 0"/>
   </xacro:widowx_arm>
   <xacro:include filename="$(find boxbot_description)/urdf/servos.urdf.xacro"/>
-  <!--xacro:include filename="$(find boxbot_description)/urdf/joint_mimic.gazebo"/-->
   <xacro:include filename="$(find boxbot_description)/urdf/materials.gazebo"/>
 </robot>
