Commit message: Use ROS node to perform joint mimicking (mimic plugin has issues in Gazebo 7.9).

File: boxbot_description/robots/boxbot.urdf.xacro (robot description, xacro)
@@ -55,5 +55,5 @@
   </xacro:widowx_arm>
   <xacro:include filename="$(find boxbot_description)/urdf/servos.urdf.xacro"/>
-  <xacro:include filename="$(find boxbot_description)/urdf/joint_mimic.gazebo"/>
+  <!--xacro:include filename="$(find boxbot_description)/urdf/joint_mimic.gazebo"/-->
   <xacro:include filename="$(find boxbot_description)/urdf/materials.gazebo"/>
 </robot>

File: boxbot_description/urdf/servos.urdf.xacro (robot description, xacro)
@@ -69,4 +69,14 @@
     </actuator>
   </transmission>
+  <transmission name="ltran7">
+    <type>transmission_interface/SimpleTransmission</type>
+    <joint name="left_gripper_prismatic_joint_2">
+      <hardwareInterface>hardware_interface/PositionJointInterface</hardwareInterface>
+    </joint>
+    <actuator name="left_motor7">
+      <hardwareInterface>hardware_interface/PositionJointInterface</hardwareInterface>
+      <mechanicalReduction>1</mechanicalReduction>
+    </actuator>
+  </transmission>
   <!--right-->
   <transmission name="rtran1">
@@ -130,3 +140,13 @@
     </actuator>
   </transmission>
+  <transmission name="rtran7">
+    <type>transmission_interface/SimpleTransmission</type>
+    <joint name="right_gripper_prismatic_joint_2">
+      <hardwareInterface>hardware_interface/PositionJointInterface</hardwareInterface>
+    </joint>
+    <actuator name="right_motor7">
+      <hardwareInterface>hardware_interface/PositionJointInterface</hardwareInterface>
+      <mechanicalReduction>1</mechanicalReduction>
+    </actuator>
+  </transmission>
 </robot>

Commit message: Update link center of masses and moments of inertia.

File: boxbot_description/robots/boxbot.urdf.xacro (robot description, xacro)
@@ -13,5 +13,5 @@
     <inertial>
       <!--placeholders-->
-      <origin xyz="0.1524 0.1524 0.009525" rpy="0 0 0"/>
+      <origin xyz="0.0 0.0 0.0" rpy="0 0 0"/>
       <mass value="1"/>
       <inertia ixx="1.0" ixy="0.0" ixz="0.0" iyy="1.0" iyz="0.0" izz="1.0"/>
@@ -32,5 +32,5 @@
     <inertial>
       <!--placeholders-->
-      <origin xyz="0.098425 0.060325 0.1778" rpy="0 0 0"/>
+      <origin xyz="0.0 0.0 0.0" rpy="0 0 0"/>
       <mass value="1"/>
       <inertia ixx="1.0" ixy="0.0" ixz="0.0" iyy="1.0" iyz="0.0" izz="1.0"/>

File: boxbot_description/urdf/widowx.urdf.xacro (robot description, xacro)
@@ -21,5 +21,5 @@
          </collision>
          <inertial>
-            <origin xyz="0 0 0" rpy="0 0 0" />
+            <origin xyz="0 0 0.0275" rpy="0 0 0" />
             <mass value="1" />
             <inertia ixx="1.0" ixy="0.0" ixz="0.0" iyy="1.0" iyz="0.0" izz="1.0" />
@@ -41,7 +41,8 @@
          </collision>
          <inertial>
-            <origin xyz="0 0 0" rpy="0 0 0" />
+            <!--estimated CM-->
+            <origin xyz="0.0 0.0 -0.04" rpy="0 0 0" />
             <mass value="0.061" />
-            <inertia ixx="1.0" ixy="0.0" ixz="0.0" iyy="1.0" iyz="0.0" izz="1.0" />
+            <inertia ixx="0.001" ixy="0.0" ixz="0.0" iyy="0.001" iyz="0.0" izz="0.001" />
          </inertial>
       </link>
@@ -61,7 +62,7 @@
          </collision>
          <inertial>
-            <origin xyz="0 0 0" rpy="0 0 0" />
+            <origin xyz="0.006670 0.0 0.083394" rpy="0 0 0" />
             <mass value="3.62e-1" />
-            <inertia ixx="1.0" ixy="0.0" ixz="0.0" iyy="1.0" iyz="0.0" izz="1.0" />
+            <inertia ixx="0.001" ixy="0.0" ixz="0.0" iyy="0.001" iyz="0.0" izz="0.001" />
          </inertial>
       </link>
@@ -81,7 +82,7 @@
          </collision>
          <inertial>
-            <origin xyz="0 0 0" rpy="0 0 0" />
+            <origin xyz="0.000018 0.0 0.090995" rpy="0 0 0" />
             <mass value="1.87e-1" />
-            <inertia ixx="1.0" ixy="0.0" ixz="0.0" iyy="1.0" iyz="0.0" izz="1.0"/>
+            <inertia ixx="0.001" ixy="0.0" ixz="0.0" iyy="0.001" iyz="0.0" izz="0.001" />
          </inertial>
       </link>
@@ -101,7 +102,7 @@
          </collision>
          <inertial>
-            <origin xyz="0 0 0" rpy="0 0 0" />
+            <origin xyz="-0.010852 0.0 0.048078" rpy="0 0 0" />
             <mass value="9.1e-2" />
-            <inertia ixx="1.0" ixy="0.0" ixz="0.0" iyy="1.0" iyz="0.0" izz="1.0" />
+            <inertia ixx="0.001" ixy="0.0" ixz="0.0" iyy="0.001" iyz="0.0" izz="0.001" />
          </inertial>
       </link>
@@ -121,7 +122,8 @@
          </collision>
          <inertial>
-            <origin xyz="0 0 0" rpy="0 0 0" />
+            <!--estimated CM-->
+            <origin xyz="-0.018000 0.0 0.01500 " rpy="0 0 0" />
             <mass value="6.3e-2" />
-            <inertia ixx="1.0" ixy="0.0" ixz="0.0" iyy="1.0" iyz="0.0" izz="1.0" />
+            <inertia ixx="0.001" ixy="0.0" ixz="0.0" iyy="0.001" iyz="0.0" izz="0.001" />
          </inertial>
       </link>

File: boxbot_description/urdf/widowx_gripper.xacro (robot description, xacro)
@@ -19,5 +19,5 @@
          <origin xyz="0 0 0" rpy="0 0 0" />
          <mass value="7.0e-3" />
-         <inertia ixx="1.0" ixy="0.0" ixz="0.0" iyy="1.0" iyz="0.0" izz="1.0" />
+         <inertia ixx="0.001" ixy="0.0" ixz="0.0" iyy="0.001" iyz="0.0" izz="0.001" />
       </inertial>
    </link>
@@ -39,7 +39,7 @@
       </collision>
       <inertial>
-         <origin xyz="0 0 0" rpy="0 0 0" />
+         <origin xyz="0.0 -0.008292 0.017304" rpy="0 0 0" />
          <mass value="8.0e-3" />
-         <inertia ixx="1.0" ixy="0.0" ixz="0.0" iyy="1.0" iyz="0.0" izz="1.0" />
+         <inertia ixx="0.001" ixy="0.0" ixz="0.0" iyy="0.001" iyz="0.0" izz="0.001" />
       </inertial>
    </link>
@@ -59,7 +59,7 @@
       </collision>
       <inertial>
-         <origin xyz="0 0 0" rpy="0 0 0" />
+         <origin xyz="0.0 0.008292 0.017304" rpy="0 0 0" />
          <mass value="8.0e-3" />
-         <inertia ixx="1.0" ixy="0.0" ixz="0.0" iyy="1.0" iyz="0.0" izz="1.0" />
+         <inertia ixx="0.001" ixy="0.0" ixz="0.0" iyy="0.001" iyz="0.0" izz="0.001" />
       </inertial>
    </link>
