Commit message: Add fixed test blocks with force sensors to the scenarios in a new URDF model.

File: boxbot_description/robots/boxbot_test_block.urdf (robot description, URDF)
Before this commit: robot boxbot, 21 links, 20 joints
Links:
- added link left_test_block, mass 0.025; collision box size=0.0762 0.01905 0.0762; visual box size=0.0762 0.01905 0.0762
- added link right_test_block, mass 0.025; collision box size=0.0762 0.01905 0.0762; visual box size=0.0762 0.01905 0.0762
Joints:
- added joint left_test_block_joint: type fixed, parent left_wrist_2_link, child left_test_block, origin xyz=0.0 0.0 0.0889
- added joint right_test_block_joint: type fixed, parent right_wrist_2_link, child right_test_block, origin xyz=0.0 0.0 0.0889

File: boxbot_gazebo/models/block_1.urdf.xacro (robot description, xacro)
@@ -21,6 +21,6 @@
   </link>
   <gazebo reference="link_1">
-    <mu1>500.0</mu1>
-    <mu2>500.0</mu2>
+    <mu1>1.0</mu1>
+    <mu2>1.0</mu2>
     <material>Gazebo/Wood</material>
   </gazebo>
