Commit message: Update ROS controllers and Gazebo functionality.

File: boxbot_description/robots/boxbot_2.urdf (robot description, URDF)
Before this commit: robot boxbot, 8 links, 2 joints
Links:
- added link left_arm_base_link; visual cylinder length=0.001 radius=.001
- added link left_gripper_1_link, mass 8.0e-3; collision mesh filename=package://boxbot_description/meshes/gripper_hand_fixed_link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; visual mesh filename=package://boxbot_description/meshes/gripper_hand_fixed_link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
- added link left_gripper_2_link, mass 8.0e-3; collision mesh filename=package://boxbot_description/meshes/gripper_hand_fixed_link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; visual mesh filename=package://boxbot_description/meshes/gripper_hand_fixed_link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
- added link left_gripper_rail_link, mass 7.0e-3; visual mesh filename=package://boxbot_description/meshes/gripper_rail_link.stl
- added link right_arm_base_link; visual cylinder length=0.001 radius=.001
- added link right_biceps_link, mass 3.62e-1; collision mesh filename=package://boxbot_description/meshes/biceps_new_link.stl; visual mesh filename=package://boxbot_description/meshes/biceps_new_link.stl
- added link right_forearm_1_link, mass 1.87e-1; collision mesh filename=package://boxbot_description/meshes/forearm_1_link.stl; visual mesh filename=package://boxbot_description/meshes/forearm_1_link.stl
- added link right_forearm_2_link, mass 1.87e-1; collision mesh filename=package://boxbot_description/meshes/forearm_2_link.stl; visual mesh filename=package://boxbot_description/meshes/forearm_2_link.stl
- added link right_gripper_1_link, mass 8.0e-3; collision mesh filename=package://boxbot_description/meshes/gripper_hand_fixed_link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; visual mesh filename=package://boxbot_description/meshes/gripper_hand_fixed_link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
- added link right_gripper_2_link, mass 8.0e-3; collision mesh filename=package://boxbot_description/meshes/gripper_hand_fixed_link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; visual mesh filename=package://boxbot_description/meshes/gripper_hand_fixed_link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
- added link right_gripper_rail_link, mass 7.0e-3; visual mesh filename=package://boxbot_description/meshes/gripper_rail_link.stl
- added link right_shoulder_link, mass 0.061; collision mesh filename=package://boxbot_description/meshes/shoulder_link.stl; visual mesh filename=package://boxbot_description/meshes/shoulder_link.stl
- added link right_wrist_1_link, mass 9.1e-2; collision mesh filename=package://boxbot_description/meshes/wrist_1_link.stl; visual mesh filename=package://boxbot_description/meshes/wrist_1_link.stl
- added link right_wrist_2_link, mass 6.3e-2; collision mesh filename=package://boxbot_description/meshes/wrist_2_link.new.stl; visual mesh filename=package://boxbot_description/meshes/wrist_2_link.new.stl
- link left_biceps_link: geometry collision mesh filename=package://boxbot_description/meshes/biceps_new_link.stl; visual mesh filename=package://boxbot_description/meshes/biceps_new_link.stl
- link torso: geometry collision mesh filename=package://boxbot_description/meshes/torso_link.stl; visual mesh filename=package://boxbot_description/meshes/torso_link.stl
Joints:
- added joint left_arm_base_joint: type fixed, parent torso, child left_arm_base_link, origin xyz=0 0.099613 0.24953 rpy=-1.570795 0 0
- added joint left_elbow_joint: type revolute, parent left_biceps_link, child left_forearm_1_link, origin xyz=-0.04825 0 0.1418 rpy=0 1.570795 3.14159, axis 0 -1 0, limit lower=-1.571 upper=1.571 effort=6 velocity=1.571
- added joint left_gripper_joint: type prismatic, parent left_gripper_rail_link, child left_gripper_1_link, origin xyz=0 0 0 rpy=0 0 0, axis 0 -1 0, limit lower=0.002 upper=0.031 effort=0 velocity=0.5
- added joint left_gripper_prismatic_joint_2: type prismatic, parent left_gripper_rail_link, child left_gripper_2_link, origin xyz=0 0 0 rpy=0 0 0, axis 0 1 0, limit lower=0.002 upper=0.031 effort=0 velocity=0.5, mimic joint=left_gripper_joint
- added joint left_joint_6: type fixed, parent left_wrist_2_link, child left_gripper_rail_link, origin xyz=0 0 0.043 rpy=0 0 0
- added joint left_shoulder_joint_2: type revolute, parent left_shoulder_link, child left_biceps_link, origin xyz=0 0 0 rpy=0 0 3.14159, axis 0 1 0, limit lower=-1.571 upper=1.571 effort=6 velocity=1.571
- added joint left_wrist_joint_1: type revolute, parent left_forearm_1_link, child left_forearm_2_link, origin xyz=0 0 0.0928 rpy=0 0 -1.570795, axis 0 0 1, limit lower=-1.745 upper=1.745 effort=6 velocity=1.571
- added joint left_wrist_joint_2: type revolute, parent left_forearm_2_link, child left_wrist_1_link, origin xyz=0 0 0.048 rpy=0 0 1.570795, axis 0 1 0, limit lower=-1.571 upper=1.571 effort=6 velocity=1.571
- added joint left_wrist_joint_3: type revolute, parent left_wrist_1_link, child left_wrist_2_link, origin xyz=0 0 0.0715 rpy=0 0 0, axis 0 0 1, limit lower=-2.617 upper=2.617 effort=6 velocity=1.571
- added joint right_arm_base_joint: type fixed, parent torso, child right_arm_base_link, origin xyz=0 -0.099613 0.24953 rpy=1.570795 0 0
- added joint right_elbow_joint: type revolute, parent right_biceps_link, child right_forearm_1_link, origin xyz=-0.04825 0 0.1418 rpy=0 1.570795 3.14159, axis 0 -1 0, limit lower=-1.571 upper=1.571 effort=6 velocity=1.571
- added joint right_gripper_joint: type prismatic, parent right_gripper_rail_link, child right_gripper_1_link, origin xyz=0 0 0 rpy=0 0 0, axis 0 -1 0, limit lower=0.002 upper=0.031 effort=0 velocity=0.5
- added joint right_gripper_prismatic_joint_2: type prismatic, parent right_gripper_rail_link, child right_gripper_2_link, origin xyz=0 0 0 rpy=0 0 0, axis 0 1 0, limit lower=0.002 upper=0.031 effort=0 velocity=0.5, mimic joint=right_gripper_joint
- added joint right_joint_6: type fixed, parent right_wrist_2_link, child right_gripper_rail_link, origin xyz=0 0 0.043 rpy=0 0 0
- added joint right_shoulder_joint_1: type revolute, parent right_arm_base_link, child right_shoulder_link, origin xyz=0 0 0 rpy=0 0 0, axis 0 0 1, limit lower=-2.617 upper=2.617 effort=6 velocity=0.785
- added joint right_shoulder_joint_2: type revolute, parent right_shoulder_link, child right_biceps_link, origin xyz=0 0 0 rpy=0 0 3.14159, axis 0 1 0, limit lower=-1.571 upper=1.571 effort=6 velocity=1.571
- added joint right_wrist_joint_1: type revolute, parent right_forearm_1_link, child right_forearm_2_link, origin xyz=0 0 0.0928 rpy=0 0 -1.570795, axis 0 0 1, limit lower=-1.745 upper=1.745 effort=6 velocity=1.571
- added joint right_wrist_joint_2: type revolute, parent right_forearm_2_link, child right_wrist_1_link, origin xyz=0 0 0.048 rpy=0 0 1.570795, axis 0 1 0, limit lower=-1.571 upper=1.571 effort=6 velocity=1.571
- added joint right_wrist_joint_3: type revolute, parent right_wrist_1_link, child right_wrist_2_link, origin xyz=0 0 0.0715 rpy=0 0 0, axis 0 0 1, limit lower=-2.617 upper=2.617 effort=6 velocity=1.571
- joint fixed: origin xyz=0 0 0.009525 rpy=0 0 0 -> xyz=0 0 0 rpy=0 0 0
- joint left_shoulder_joint_1: origin xyz=0.099613 0 0.243180 rpy=0 0 0 -> xyz=0 0 0 rpy=0 0 0; parent torso -> left_arm_base_link

File: boxbot_description/urdf/servos.urdf.xacro (robot description, xacro)
@@ -11,5 +11,5 @@
   <transmission name="ltran1">
     <type>transmission_interface/SimpleTransmission</type>
-    <joint name="left_joint_1">
+    <joint name="left_shoulder_joint_1">
       <hardwareInterface>hardware_interface/PositionJointInterface</hardwareInterface>
     </joint>
@@ -21,5 +21,5 @@
   <transmission name="ltran2">
     <type>transmission_interface/SimpleTransmission</type>
-    <joint name="left_joint_2">
+    <joint name="left_shoulder_joint_2">
       <hardwareInterface>hardware_interface/PositionJointInterface</hardwareInterface>
     </joint>
@@ -31,5 +31,5 @@
   <transmission name="ltran3">
     <type>transmission_interface/SimpleTransmission</type>
-    <joint name="left_joint_3">
+    <joint name="left_elbow_joint">
       <hardwareInterface>hardware_interface/PositionJointInterface</hardwareInterface>
     </joint>
@@ -41,5 +41,5 @@
   <transmission name="ltran4">
     <type>transmission_interface/SimpleTransmission</type>
-    <joint name="left_joint_4">
+    <joint name="left_wrist_joint_1">
       <hardwareInterface>hardware_interface/PositionJointInterface</hardwareInterface>
     </joint>
@@ -51,5 +51,5 @@
   <transmission name="ltran5">
     <type>transmission_interface/SimpleTransmission</type>
-    <joint name="left_joint_5">
+    <joint name="left_wrist_joint_2">
       <hardwareInterface>hardware_interface/PositionJointInterface</hardwareInterface>
     </joint>
@@ -61,5 +61,5 @@
   <transmission name="ltran6">
     <type>transmission_interface/SimpleTransmission</type>
-    <joint name="left_gripper_joint">
+    <joint name="left_wrist_joint_3">
       <hardwareInterface>hardware_interface/PositionJointInterface</hardwareInterface>
     </joint>
@@ -71,5 +71,5 @@
   <transmission name="ltran7">
     <type>transmission_interface/SimpleTransmission</type>
-    <joint name="left_gripper_prismatic_joint_2">
+    <joint name="left_gripper_joint">
       <hardwareInterface>hardware_interface/PositionJointInterface</hardwareInterface>
     </joint>
@@ -79,8 +79,18 @@
     </actuator>
   </transmission>
+  <transmission name="ltran8">
+    <type>transmission_interface/SimpleTransmission</type>
+    <joint name="left_gripper_prismatic_joint_2">
+      <hardwareInterface>hardware_interface/PositionJointInterface</hardwareInterface>
+    </joint>
+    <actuator name="left_motor8">
+      <hardwareInterface>hardware_interface/PositionJointInterface</hardwareInterface>
+      <mechanicalReduction>1</mechanicalReduction>
+    </actuator>
+  </transmission>
   <!--right-->
   <transmission name="rtran1">
     <type>transmission_interface/SimpleTransmission</type>
-    <joint name="right_joint_1">
+    <joint name="right_shoulder_joint_1">
       <hardwareInterface>hardware_interface/PositionJointInterface</hardwareInterface>
     </joint>
@@ -92,5 +102,5 @@
   <transmission name="rtran2">
     <type>transmission_interface/SimpleTransmission</type>
-    <joint name="right_joint_2">
+    <joint name="right_shoulder_joint_2">
       <hardwareInterface>hardware_interface/PositionJointInterface</hardwareInterface>
     </joint>
@@ -102,5 +112,5 @@
   <transmission name="rtran3">
     <type>transmission_interface/SimpleTransmission</type>
-    <joint name="right_joint_3">
+    <joint name="right_elbow_joint">
       <hardwareInterface>hardware_interface/PositionJointInterface</hardwareInterface>
     </joint>
@@ -112,5 +122,5 @@
   <transmission name="rtran4">
     <type>transmission_interface/SimpleTransmission</type>
-    <joint name="right_joint_4">
+    <joint name="right_wrist_joint_1">
       <hardwareInterface>hardware_interface/PositionJointInterface</hardwareInterface>
     </joint>
@@ -122,5 +132,5 @@
   <transmission name="rtran5">
     <type>transmission_interface/SimpleTransmission</type>
-    <joint name="right_joint_5">
+    <joint name="right_wrist_joint_2">
       <hardwareInterface>hardware_interface/PositionJointInterface</hardwareInterface>
     </joint>
@@ -132,5 +142,5 @@
   <transmission name="rtran6">
     <type>transmission_interface/SimpleTransmission</type>
-    <joint name="right_gripper_joint">
+    <joint name="right_wrist_joint_3">
       <hardwareInterface>hardware_interface/PositionJointInterface</hardwareInterface>
     </joint>
@@ -142,5 +152,5 @@
   <transmission name="rtran7">
     <type>transmission_interface/SimpleTransmission</type>
-    <joint name="right_gripper_prismatic_joint_2">
+    <joint name="right_gripper_joint">
       <hardwareInterface>hardware_interface/PositionJointInterface</hardwareInterface>
     </joint>
@@ -150,3 +160,13 @@
     </actuator>
   </transmission>
+  <transmission name="rtran8">
+    <type>transmission_interface/SimpleTransmission</type>
+    <joint name="right_gripper_prismatic_joint_2">
+      <hardwareInterface>hardware_interface/PositionJointInterface</hardwareInterface>
+    </joint>
+    <actuator name="right_motor8">
+      <hardwareInterface>hardware_interface/PositionJointInterface</hardwareInterface>
+      <mechanicalReduction>1</mechanicalReduction>
+    </actuator>
+  </transmission>
 </robot>

File: boxbot_description/urdf/widowx_6dof.urdf.xacro (robot description, xacro)
@@ -6,5 +6,11 @@
    <xacro:macro name="widowx_arm" params="parent prefix *origin">
       <!-- links -->
-      <link name="${prefix}arm_base_link"/>
+      <link name="${prefix}arm_base_link">
+         <inertial>
+            <origin xyz="0.0 0.0 -0.04" rpy="0 0 0" />
+            <mass value="0.001" />
+            <inertia ixx="0.001" ixy="0.0" ixz="0.0" iyy="0.001" iyz="0.0" izz="0.001" />
+         </inertial>
+      </link>
       <link name="${prefix}shoulder_link">
          <visual>

File: boxbot_description/urdf/widowx_gripper.xacro (robot description, xacro)
@@ -22,6 +22,4 @@
       </inertial>
    </link>
-   <!--link name="${prefix}gripper_aux_link">
-   </link-->
    <link name="${prefix}gripper_1_link">
       <visual>

Commit message: Update some various parameters.

File: boxbot_description/robots/boxbot_2.urdf (robot description, URDF)
Before this commit: robot boxbot, 22 links, 21 joints
Links:
- link left_arm_base_link: mass None -> 0.001; geometry 
- link right_arm_base_link: mass None -> 0.001; geometry 
Joints:
- joint left_wrist_joint_1: limit lower=-1.745 upper=1.745 effort=6 velocity=1.571 -> lower=-2.617 upper=2.617 effort=2.5 velocity=1.571
- joint left_wrist_joint_2: limit lower=-1.571 upper=1.571 effort=6 velocity=1.571 -> lower=-1.745 upper=1.745 effort=2.5 velocity=1.571
- joint left_wrist_joint_3: limit lower=-2.617 upper=2.617 effort=6 velocity=1.571 -> lower=-2.617 upper=2.617 effort=1.5 velocity=1.571
- joint right_wrist_joint_1: limit lower=-1.745 upper=1.745 effort=6 velocity=1.571 -> lower=-2.617 upper=2.617 effort=2.5 velocity=1.571
- joint right_wrist_joint_2: limit lower=-1.571 upper=1.571 effort=6 velocity=1.571 -> lower=-1.745 upper=1.745 effort=2.5 velocity=1.571
- joint right_wrist_joint_3: limit lower=-2.617 upper=2.617 effort=6 velocity=1.571 -> lower=-2.617 upper=2.617 effort=1.5 velocity=1.571

File: boxbot_description/urdf/widowx_6dof.urdf.xacro (robot description, xacro)
@@ -165,5 +165,5 @@
          <child link="${prefix}forearm_2_link" />
          <axis xyz="0 0 1" />
-         <limit lower="-1.745" upper="1.745" effort="6" velocity="1.571" />
+         <limit lower="-2.617" upper="2.617" effort="2.5" velocity="1.571" />
       </joint>
       <joint name="${prefix}wrist_joint_2" type="revolute">
@@ -172,5 +172,5 @@
          <child link="${prefix}wrist_1_link" />
          <axis xyz="0 1 0" />
-         <limit lower="-1.571" upper="1.571" effort="6" velocity="1.571" />
+         <limit lower="-1.745" upper="1.745" effort="2.5" velocity="1.571" />
       </joint>
       <joint name="${prefix}wrist_joint_3" type="revolute">
@@ -179,5 +179,5 @@
          <child link="${prefix}wrist_2_link" />
          <axis xyz="0 0 1" />
-         <limit lower="-2.617" upper="2.617" effort="6" velocity="1.571" />
+         <limit lower="-2.617" upper="2.617" effort="1.5" velocity="1.571" />
       </joint>
       <!-- gripper -->
