Commit message: General cleanup of repository.

File: boxbot_description/robots/boxbot_5dof.urdf (robot description, URDF)
Before this commit: robot boxbot, 21 links, 20 joints
Links:
- removed link base_link
- removed link left_forearm_link
- removed link right_forearm_link
- added link left_forearm_1_link, mass 1.87e-1; collision mesh filename=package://boxbot_description/meshes/forearm_link.new.stl; visual mesh filename=package://boxbot_description/meshes/forearm_link.new.stl
- added link right_forearm_1_link, mass 1.87e-1; collision mesh filename=package://boxbot_description/meshes/forearm_link.new.stl; visual mesh filename=package://boxbot_description/meshes/forearm_link.new.stl
- link left_arm_base_link: mass 1 -> 0.001; geometry 
- link right_arm_base_link: mass 1 -> 0.001; geometry 
- link torso: geometry collision mesh filename=package://boxbot_description/meshes/torso_link.stl; visual mesh filename=package://boxbot_description/meshes/torso_link.stl
Joints:
- removed joint left_joint_6
- removed joint right_joint_6
- removed joint waist_joint
- added joint left__rail_joint: type fixed, parent left_wrist_2_link, child left_gripper_rail_link, origin xyz=0 0 0.043 rpy=0 0 0
- added joint right__rail_joint: type fixed, parent right_wrist_2_link, child right_gripper_rail_link, origin xyz=0 0 0.043 rpy=0 0 0
- joint fixed: child base_link -> torso; origin xyz=0 0 0.009525 rpy=0 0 0 -> xyz=0 0 0 rpy=0 0 0
- joint left_arm_base_joint: origin xyz=0 0.087325 0.0635 rpy=-1.5707963268 0 0 -> xyz=0 0.099613 0.24953 rpy=-1.570795 0 0
- joint left_joint_1: origin xyz=0 0 0.065 rpy=0 0 0 -> xyz=0 0 0 rpy=0 0 0
- joint left_joint_3: child left_forearm_link -> left_forearm_1_link
- joint left_joint_4: parent left_forearm_link -> left_forearm_1_link
- joint right_arm_base_joint: origin xyz=0 -0.087325 0.0635 rpy=1.5707963268 0 0 -> xyz=0 -0.099613 0.24953 rpy=1.570795 0 0
- joint right_joint_1: origin xyz=0 0 0.065 rpy=0 0 0 -> xyz=0 0 0 rpy=0 0 0
- joint right_joint_3: child right_forearm_link -> right_forearm_1_link
- joint right_joint_4: parent right_forearm_link -> right_forearm_1_link

File: boxbot_description/robots/boxbot_5dof.urdf.xacro (robot description, xacro)
@@ -1,31 +1,19 @@
 <?xml version="1.0"?>
 <robot name="boxbot" xmlns:xacro="http://ros.org/wiki/xacro">
+  <xacro:property name="M_SCALE" value="0.001"/>
   <xacro:include filename="$(find boxbot_description)/urdf/common_materials.xacro" />
   <link name="world"/>
-  <link name="base_link">
-    <visual>
-      <geometry>
-        <box size="0.3048 0.3048 0.01905"/>
-      </geometry>
-      <xacro:material_yellow/>
-    </visual>
-    <!--Can't get collision to work for this link; likely a collision issue with the torso.-->
-    <inertial>
-      <!--placeholders-->
-      <origin xyz="0.0 0.0 0.0" rpy="0 0 0"/>
-      <mass value="1"/>
-      <inertia ixx="1.0" ixy="0.0" ixz="0.0" iyy="1.0" iyz="0.0" izz="1.0"/>
-    </inertial>
-  </link>
   <link name="torso">
     <visual>
+      <origin xyz="0 0 0" rpy="1.5707963268 0 1.5707963268" />
       <geometry>
-        <box size="0.19685 0.12065 0.3556"/>
+        <mesh filename="package://boxbot_description/meshes/torso_link.stl"/>
       </geometry>
       <xacro:material_yellow/>
     </visual>
     <collision>
+      <origin xyz="0 0 0" rpy="1.5707963268 0 1.5707963268" />
       <geometry>
-        <box size="0.19685 0.12065 0.3556"/>
+        <mesh filename="package://boxbot_description/meshes/torso_link.stl"/>
       </geometry>
     </collision>
@@ -38,22 +26,19 @@
   </link>
   <joint name="fixed" type="fixed">
-    <origin xyz="0 0 0.009525" rpy="0 0 0"/>
+    <origin xyz="0 0 0" rpy="0 0 0"/>
     <parent link="world"/>
-    <child link="base_link"/>
-  </joint>
-  <joint name="waist_joint" type="fixed">
-    <origin xyz="0 0 0.187325" rpy="0 0 0"/>
-    <parent link="base_link"/>
     <child link="torso"/>
   </joint>
   <xacro:include filename="$(find boxbot_description)/urdf/widowx.urdf.xacro"/>
   <xacro:widowx_arm parent="torso" prefix="left_">
-    <origin xyz="0 0.087325 0.0635" rpy="-1.5707963268 0 0"/>
+    <origin xyz="0 ${M_SCALE*99.613} ${M_SCALE*249.53}" rpy="-${M_PI/2.0} 0 0" />
   </xacro:widowx_arm>
   <xacro:include filename="$(find boxbot_description)/urdf/widowx.urdf.xacro"/>
   <xacro:widowx_arm parent="torso" prefix="right_">
-    <origin xyz="0 -0.087325 0.0635" rpy="1.5707963268 0 0"/>
+    <origin xyz="0 -${M_SCALE*99.613} ${M_SCALE*249.53}" rpy="${M_PI/2.0} 0 0"/>
   </xacro:widowx_arm>
   <xacro:include filename="$(find boxbot_description)/urdf/servos.urdf.xacro"/>
+  <xacro:ros_control_widowx six_dof="false"/>
   <xacro:include filename="$(find boxbot_description)/urdf/materials.gazebo"/>
+  <xacro:gazebo_widowx six_dof="false"/>
 </robot>

File: boxbot_description/robots/boxbot_6dof.urdf (robot description, URDF)
Before this commit: robot boxbot, 22 links, 21 joints
Joints:
- removed joint left_elbow_joint
- removed joint left_shoulder_joint_1
- removed joint left_shoulder_joint_2
- removed joint left_wrist_joint_1
- removed joint left_wrist_joint_2
- removed joint left_wrist_joint_3
- removed joint right_elbow_joint
- removed joint right_shoulder_joint_1
- removed joint right_shoulder_joint_2
- removed joint right_wrist_joint_1
- removed joint right_wrist_joint_2
- removed joint right_wrist_joint_3
- added joint left__rail_joint: type fixed, parent left_wrist_2_link, child left_gripper_rail_link, origin xyz=0 0 0.043 rpy=0 0 0
- added joint left_joint_1: type revolute, parent left_arm_base_link, child left_shoulder_link, origin xyz=0 0 0 rpy=0 0 0, axis 0 0 1, limit lower=-2.617 upper=2.617 effort=6 velocity=0.785
- added joint left_joint_2: type revolute, parent left_shoulder_link, child left_biceps_link, origin xyz=0 0 0 rpy=0 0 3.14159, axis 0 1 0, limit lower=-1.571 upper=1.571 effort=6 velocity=1.571
- added joint left_joint_3: type revolute, parent left_biceps_link, child left_forearm_1_link, origin xyz=-0.04825 0 0.1418 rpy=0 1.570795 3.14159, axis 0 -1 0, limit lower=-1.571 upper=1.571 effort=6 velocity=1.571
- added joint left_joint_4: type revolute, parent left_forearm_1_link, child left_forearm_2_link, origin xyz=0 0 0.0928 rpy=0 0 -1.570795, axis 0 0 1, limit lower=-2.617 upper=2.617 effort=2.5 velocity=1.571
- added joint left_joint_5: type revolute, parent left_forearm_2_link, child left_wrist_1_link, origin xyz=0 0 0.048 rpy=0 0 1.570795, axis 0 1 0, limit lower=-1.745 upper=1.745 effort=2.5 velocity=1.571
- added joint right__rail_joint: type fixed, parent right_wrist_2_link, child right_gripper_rail_link, origin xyz=0 0 0.043 rpy=0 0 0
- added joint right_joint_1: type revolute, parent right_arm_base_link, child right_shoulder_link, origin xyz=0 0 0 rpy=0 0 0, axis 0 0 1, limit lower=-2.617 upper=2.617 effort=6 velocity=0.785
- added joint right_joint_2: type revolute, parent right_shoulder_link, child right_biceps_link, origin xyz=0 0 0 rpy=0 0 3.14159, axis 0 1 0, limit lower=-1.571 upper=1.571 effort=6 velocity=1.571
- added joint right_joint_3: type revolute, parent right_biceps_link, child right_forearm_1_link, origin xyz=-0.04825 0 0.1418 rpy=0 1.570795 3.14159, axis 0 -1 0, limit lower=-1.571 upper=1.571 effort=6 velocity=1.571
- added joint right_joint_4: type revolute, parent right_forearm_1_link, child right_forearm_2_link, origin xyz=0 0 0.0928 rpy=0 0 -1.570795, axis 0 0 1, limit lower=-2.617 upper=2.617 effort=2.5 velocity=1.571
- added joint right_joint_5: type revolute, parent right_forearm_2_link, child right_wrist_1_link, origin xyz=0 0 0.048 rpy=0 0 1.570795, axis 0 1 0, limit lower=-1.745 upper=1.745 effort=2.5 velocity=1.571
- joint left_joint_6: axis (none) -> 0 0 1; child left_gripper_rail_link -> left_wrist_2_link; limit (none) -> lower=-2.617 upper=2.617 effort=1.5 velocity=1.571; origin xyz=0 0 0.043 rpy=0 0 0 -> xyz=0 0 0.0715 rpy=0 0 0; parent left_wrist_2_link -> left_wrist_1_link; type fixed -> revolute
- joint right_joint_6: axis (none) -> 0 0 1; child right_gripper_rail_link -> right_wrist_2_link; limit (none) -> lower=-2.617 upper=2.617 effort=1.5 velocity=1.571; origin xyz=0 0 0.043 rpy=0 0 0 -> xyz=0 0 0.0715 rpy=0 0 0; parent right_wrist_2_link -> right_wrist_1_link; type fixed -> revolute

File: boxbot_description/robots/boxbot_6dof.urdf.xacro (robot description, xacro)
@@ -39,4 +39,6 @@
   </xacro:widowx_arm>
   <xacro:include filename="$(find boxbot_description)/urdf/servos.urdf.xacro"/>
+  <xacro:ros_control_widowx six_dof="true"/>
   <xacro:include filename="$(find boxbot_description)/urdf/materials.gazebo"/>
+  <xacro:gazebo_widowx six_dof="true"/>
 </robot>
