Commit message: General cleanup of repository.

File: boxbot_description/urdf/servos.urdf.xacro (robot description, xacro)
@@ -1,172 +1,178 @@
 <?xml version="1.0"?>
-<robot>
-  <!--gazebo ros control-->
-  <gazebo>
-    <plugin name="gazebo_ros_control" filename="libgazebo_ros_control.so">
-      <robotNamespace>/boxbot</robotNamespace>
-    </plugin>
-  </gazebo>
-  <!--transmissions-->
-  <!--left-->
-  <transmission name="ltran1">
-    <type>transmission_interface/SimpleTransmission</type>
-    <joint name="left_shoulder_joint_1">
-      <hardwareInterface>hardware_interface/PositionJointInterface</hardwareInterface>
-    </joint>
-    <actuator name="left_motor1">
-      <hardwareInterface>hardware_interface/PositionJointInterface</hardwareInterface>
-      <mechanicalReduction>1</mechanicalReduction>
-    </actuator>
-  </transmission>
-  <transmission name="ltran2">
-    <type>transmission_interface/SimpleTransmission</type>
-    <joint name="left_shoulder_joint_2">
-      <hardwareInterface>hardware_interface/PositionJointInterface</hardwareInterface>
-    </joint>
-    <actuator name="left_motor2">
-      <hardwareInterface>hardware_interface/PositionJointInterface</hardwareInterface>
-      <mechanicalReduction>1</mechanicalReduction>
-    </actuator>
-  </transmission>
-  <transmission name="ltran3">
-    <type>transmission_interface/SimpleTransmission</type>
-    <joint name="left_elbow_joint">
-      <hardwareInterface>hardware_interface/PositionJointInterface</hardwareInterface>
-    </joint>
-    <actuator name="left_motor3">
-      <hardwareInterface>hardware_interface/PositionJointInterface</hardwareInterface>
-      <mechanicalReduction>1</mechanicalReduction>
-    </actuator>
-  </transmission>
-  <transmission name="ltran4">
-    <type>transmission_interface/SimpleTransmission</type>
-    <joint name="left_wrist_joint_1">
-      <hardwareInterface>hardware_interface/PositionJointInterface</hardwareInterface>
-    </joint>
-    <actuator name="left_motor4">
-      <hardwareInterface>hardware_interface/PositionJointInterface</hardwareInterface>
-      <mechanicalReduction>1</mechanicalReduction>
-    </actuator>
-  </transmission>
-  <transmission name="ltran5">
-    <type>transmission_interface/SimpleTransmission</type>
-    <joint name="left_wrist_joint_2">
-      <hardwareInterface>hardware_interface/PositionJointInterface</hardwareInterface>
-    </joint>
-    <actuator name="left_motor5">
-      <hardwareInterface>hardware_interface/PositionJointInterface</hardwareInterface>
-      <mechanicalReduction>1</mechanicalReduction>
-    </actuator>
-  </transmission>
-  <transmission name="ltran6">
-    <type>transmission_interface/SimpleTransmission</type>
-    <joint name="left_wrist_joint_3">
-      <hardwareInterface>hardware_interface/PositionJointInterface</hardwareInterface>
-    </joint>
-    <actuator name="left_motor6">
-      <hardwareInterface>hardware_interface/PositionJointInterface</hardwareInterface>
-      <mechanicalReduction>1</mechanicalReduction>
-    </actuator>
-  </transmission>
-  <transmission name="ltran7">
-    <type>transmission_interface/SimpleTransmission</type>
-    <joint name="left_gripper_joint">
-      <hardwareInterface>hardware_interface/PositionJointInterface</hardwareInterface>
-    </joint>
-    <actuator name="left_motor7">
-      <hardwareInterface>hardware_interface/PositionJointInterface</hardwareInterface>
-      <mechanicalReduction>1</mechanicalReduction>
-    </actuator>
-  </transmission>
-  <transmission name="ltran8">
-    <type>transmission_interface/SimpleTransmission</type>
-    <joint name="left_gripper_prismatic_joint_2">
-      <hardwareInterface>hardware_interface/PositionJointInterface</hardwareInterface>
-    </joint>
-    <actuator name="left_motor8">
-      <hardwareInterface>hardware_interface/PositionJointInterface</hardwareInterface>
-      <mechanicalReduction>1</mechanicalReduction>
-    </actuator>
-  </transmission>
-  <!--right-->
-  <transmission name="rtran1">
-    <type>transmission_interface/SimpleTransmission</type>
-    <joint name="right_shoulder_joint_1">
-      <hardwareInterface>hardware_interface/PositionJointInterface</hardwareInterface>
-    </joint>
-    <actuator name="right_motor1">
-      <hardwareInterface>hardware_interface/PositionJointInterface</hardwareInterface>
-      <mechanicalReduction>1</mechanicalReduction>
-    </actuator>
-  </transmission>
-  <transmission name="rtran2">
-    <type>transmission_interface/SimpleTransmission</type>
-    <joint name="right_shoulder_joint_2">
-      <hardwareInterface>hardware_interface/PositionJointInterface</hardwareInterface>
-    </joint>
-    <actuator name="right_motor2">
-      <hardwareInterface>hardware_interface/PositionJointInterface</hardwareInterface>
-      <mechanicalReduction>1</mechanicalReduction>
-    </actuator>
-  </transmission>
-  <transmission name="rtran3">
-    <type>transmission_interface/SimpleTransmission</type>
-    <joint name="right_elbow_joint">
-      <hardwareInterface>hardware_interface/PositionJointInterface</hardwareInterface>
-    </joint>
-    <actuator name="right_motor3">
-      <hardwareInterface>hardware_interface/PositionJointInterface</hardwareInterface>
-      <mechanicalReduction>1</mechanicalReduction>
-    </actuator>
-  </transmission>
-  <transmission name="rtran4">
-    <type>transmission_interface/SimpleTransmission</type>
-    <joint name="right_wrist_joint_1">
-      <hardwareInterface>hardware_interface/PositionJointInterface</hardwareInterface>
-    </joint>
-    <actuator name="right_motor4">
-      <hardwareInterface>hardware_interface/PositionJointInterface</hardwareInterface>
-      <mechanicalReduction>1</mechanicalReduction>
-    </actuator>
-  </transmission>
-  <transmission name="rtran5">
-    <type>transmission_interface/SimpleTransmission</type>
-    <joint name="right_wrist_joint_2">
-      <hardwareInterface>hardware_interface/PositionJointInterface</hardwareInterface>
-    </joint>
-    <actuator name="right_motor5">
-      <hardwareInterface>hardware_interface/PositionJointInterface</hardwareInterface>
-      <mechanicalReduction>1</mechanicalReduction>
-    </actuator>
-  </transmission>
-  <transmission name="rtran6">
-    <type>transmission_interface/SimpleTransmission</type>
-    <joint name="right_wrist_joint_3">
-      <hardwareInterface>hardware_interface/PositionJointInterface</hardwareInterface>
-    </joint>
-    <actuator name="right_motor6">
-      <hardwareInterface>hardware_interface/PositionJointInterface</hardwareInterface>
-      <mechanicalReduction>1</mechanicalReduction>
-    </actuator>
-  </transmission>
-  <transmission name="rtran7">
-    <type>transmission_interface/SimpleTransmission</type>
-    <joint name="right_gripper_joint">
-      <hardwareInterface>hardware_interface/PositionJointInterface</hardwareInterface>
-    </joint>
-    <actuator name="right_motor7">
-      <hardwareInterface>hardware_interface/PositionJointInterface</hardwareInterface>
-      <mechanicalReduction>1</mechanicalReduction>
-    </actuator>
-  </transmission>
-  <transmission name="rtran8">
-    <type>transmission_interface/SimpleTransmission</type>
-    <joint name="right_gripper_prismatic_joint_2">
-      <hardwareInterface>hardware_interface/PositionJointInterface</hardwareInterface>
-    </joint>
-    <actuator name="right_motor8">
-      <hardwareInterface>hardware_interface/PositionJointInterface</hardwareInterface>
-      <mechanicalReduction>1</mechanicalReduction>
-    </actuator>
-  </transmission>
+<robot xmlns:xacro="http://ros.org/wiki/xacro">
+  <xacro:macro name="ros_control_widowx" params="six_dof">
+    <!--gazebo ros control-->
+    <gazebo>
+      <plugin name="gazebo_ros_control" filename="libgazebo_ros_control.so">
+        <robotNamespace>/boxbot</robotNamespace>
+        </plugin>
+    </gazebo>
+    <!--transmissions-->
+    <!--left-->
+    <transmission name="ltran1">
+      <type>transmission_interface/SimpleTransmission</type>
+      <joint name="left_joint_1">
+        <hardwareInterface>hardware_interface/PositionJointInterface</hardwareInterface>
+      </joint>
+      <actuator name="left_motor1">
+        <hardwareInterface>hardware_interface/PositionJointInterface</hardwareInterface>
+        <mechanicalReduction>1</mechanicalReduction>
+      </actuator>
+    </transmission>
+    <transmission name="ltran2">
+      <type>transmission_interface/SimpleTransmission</type>
+      <joint name="left_joint_2">
+        <hardwareInterface>hardware_interface/PositionJointInterface</hardwareInterface>
+      </joint>
+      <actuator name="left_motor2">
+        <hardwareInterface>hardware_interface/PositionJointInterface</hardwareInterface>
+        <mechanicalReduction>1</mechanicalReduction>
+      </actuator>
+    </transmission>
+    <transmission name="ltran3">
+      <type>transmission_interface/SimpleTransmission</type>
+      <joint name="left_joint_3">
+        <hardwareInterface>hardware_interface/PositionJointInterface</hardwareInterface>
+      </joint>
+      <actuator name="left_motor3">
+        <hardwareInterface>hardware_interface/PositionJointInterface</hardwareInterface>
+        <mechanicalReduction>1</mechanicalReduction>
+      </actuator>
+    </transmission>
+    <transmission name="ltran4">
+      <type>transmission_interface/SimpleTransmission</type>
+      <joint name="left_joint_4">
+        <hardwareInterface>hardware_interface/PositionJointInterface</hardwareInterface>
+      </joint>
+      <actuator name="left_motor4">
+        <hardwareInterface>hardware_interface/PositionJointInterface</hardwareInterface>
+        <mechanicalReduction>1</mechanicalReduction>
+      </actuator>
+    </transmission>
+    <transmission name="ltran5">
+      <type>transmission_interface/SimpleTransmission</type>
+      <joint name="left_joint_5">
+        <hardwareInterface>hardware_interface/PositionJointInterface</hardwareInterface>
+      </joint>
+      <actuator name="left_motor5">
+        <hardwareInterface>hardware_interface/PositionJointInterface</hardwareInterface>
+        <mechanicalReduction>1</mechanicalReduction>
+      </actuator>
+    </transmission>
+    <xacro:if value="${six_dof}">
+      <transmission name="ltran6">
+        <type>transmission_interface/SimpleTransmission</type>
+        <joint name="left_joint_6">
+          <hardwareInterface>hardware_interface/PositionJointInterface</hardwareInterface>
+        </joint>
+        <actuator name="left_motor6">
+          <hardwareInterface>hardware_interface/PositionJointInterface</hardwareInterface>
+          <mechanicalReduction>1</mechanicalReduction>
+        </actuator>
+      </transmission>
+    </xacro:if>
+    <transmission name="ltrang">
+      <type>transmission_interface/SimpleTransmission</type>
+      <joint name="left_gripper_joint">
+        <hardwareInterface>hardware_interface/PositionJointInterface</hardwareInterface>
+      </joint>
+      <actuator name="left_motorg">
+        <hardwareInterface>hardware_interface/PositionJointInterface</hardwareInterface>
+        <mechanicalReduction>1</mechanicalReduction>
+      </actuator>
+    </transmission>
+    <transmission name="ltrang2">
+      <type>transmission_interface/SimpleTransmission</type>
+      <joint name="left_gripper_prismatic_joint_2">
+        <hardwareInterface>hardware_interface/PositionJointInterface</hardwareInterface>
+      </joint>
+      <actuator name="left_motorg2">
+        <hardwareInterface>hardware_interface/PositionJointInterface</hardwareInterface>
+        <mechanicalReduction>1</mechanicalReduction>
+      </actuator>
+    </transmission>
+    <!--right-->
+    <transmission name="rtran1">
+      <type>transmission_interface/SimpleTransmission</type>
+      <joint name="right_joint_1">
+        <hardwareInterface>hardware_interface/PositionJointInterface</hardwareInterface>
+      </joint>
+      <actuator name="right_motor1">
+        <hardwareInterface>hardware_interface/PositionJointInterface</hardwareInterface>
+        <mechanicalReduction>1</mechanicalReduction>
+      </actuator>
+    </transmission>
+    <transmission name="rtran2">
+      <type>transmission_interface/SimpleTransmission</type>
+      <joint name="right_joint_2">
+        <hardwareInterface>hardware_interface/PositionJointInterface</hardwareInterface>
+      </joint>
+      <actuator name="right_motor2">
+        <hardwareInterface>hardware_interface/PositionJointInterface</hardwareInterface>
+        <mechanicalReduction>1</mechanicalReduction>
+      </actuator>
+    </transmission>
+    <transmission name="rtran3">
+      <type>transmission_interface/SimpleTransmission</type>
+      <joint name="right_joint_3">
+        <hardwareInterface>hardware_interface/PositionJointInterface</hardwareInterface>
+      </joint>
+      <actuator name="right_motor3">
+        <hardwareInterface>hardware_interface/PositionJointInterface</hardwareInterface>
+        <mechanicalReduction>1</mechanicalReduction>
+      </actuator>
+    </transmission>
+    <transmission name="rtran4">
+      <type>transmission_interface/SimpleTransmission</type>
+      <joint name="right_joint_4">
+        <hardwareInterface>hardware_interface/PositionJointInterface</hardwareInterface>
+      </joint>
+      <actuator name="right_motor4">
+        <hardwareInterface>hardware_interface/PositionJointInterface</hardwareInterface>
+        <mechanicalReduction>1</mechanicalReduction>
+      </actuator>
+    </transmission>
+    <transmission name="rtran5">
+      <type>transmission_interface/SimpleTransmission</type>
+      <joint name="right_joint_5">
+        <hardwareInterface>hardware_interface/PositionJointInterface</hardwareInterface>
+      </joint>
+      <actuator name="right_motor5">
+        <hardwareInterface>hardware_interface/PositionJointInterface</hardwareInterface>
+        <mechanicalReduction>1</mechanicalReduction>
+      </actuator>
+    </transmission>
+    <xacro:if value="${six_dof}">
+      <transmission name="rtran6">
+        <type>transmission_interface/SimpleTransmission</type>
+        <joint name="right_joint_6">
+          <hardwareInterface>hardware_interface/PositionJointInterface</hardwareInterface>
+        </joint>
+        <actuator name="right_motor6">
+          <hardwareInterface>hardware_interface/PositionJointInterface</hardwareInterface>
+          <mechanicalReduction>1</mechanicalReduction>
+        </actuator>
+      </transmission>
+    </xacro:if>
+    <transmission name="rtrang">
+      <type>transmission_interface/SimpleTransmission</type>
+      <joint name="right_gripper_joint">
+        <hardwareInterface>hardware_interface/PositionJointInterface</hardwareInterface>
+      </joint>
+      <actuator name="right_motorg">
+        <hardwareInterface>hardware_interface/PositionJointInterface</hardwareInterface>
+        <mechanicalReduction>1</mechanicalReduction>
+      </actuator>
+    </transmission>
+    <transmission name="rtrang2">
+      <type>transmission_interface/SimpleTransmission</type>
+      <joint name="right_gripper_prismatic_joint_2">
+        <hardwareInterface>hardware_interface/PositionJointInterface</hardwareInterface>
+      </joint>
+      <actuator name="right_motorg2">
+        <hardwareInterface>hardware_interface/PositionJointInterface</hardwareInterface>
+        <mechanicalReduction>1</mechanicalReduction>
+      </actuator>
+    </transmission>
+  </xacro:macro>
 </robot>

File: boxbot_description/urdf/widowx.urdf.xacro (robot description, xacro)
@@ -7,21 +7,8 @@
       <!-- links -->
       <link name="${prefix}arm_base_link">
-         <visual>
-            <origin xyz="0 0 0" rpy="0 0 0" />
-            <geometry>
-               <cylinder radius=".072" length="0.055"/>
-            </geometry>
-            <xacro:material_black />
-	       </visual>
-         <collision>
-            <origin xyz="0 0 0" rpy="0 0 0" />
-            <geometry>
-               <cylinder radius=".072" length="0.055"/>
-            </geometry>
-         </collision>
          <inertial>
-            <origin xyz="0 0 0.0275" rpy="0 0 0" />
-            <mass value="1" />
-            <inertia ixx="1.0" ixy="0.0" ixz="0.0" iyy="1.0" iyz="0.0" izz="1.0" />
+            <origin xyz="0.0 0.0 -0.04" rpy="0 0 0" />
+            <mass value="0.001" />
+            <inertia ixx="0.001" ixy="0.0" ixz="0.0" iyy="0.001" iyz="0.0" izz="0.001" />
          </inertial>
       </link>
@@ -66,5 +53,5 @@
          </inertial>
       </link>
-      <link name="${prefix}forearm_link">
+      <link name="${prefix}forearm_1_link">
          <visual>
             <origin xyz="0 0 0" rpy="0 0 0" />
@@ -133,5 +120,5 @@
       </joint>
       <joint name="${prefix}joint_1" type="revolute">
-         <origin xyz="0 0 0.065" rpy="0 0 0" />
+         <origin xyz="0 0 0" rpy="0 0 0" />
          <parent link="${prefix}arm_base_link" />
          <child link="${prefix}shoulder_link" />
@@ -150,5 +137,5 @@
          <origin xyz="${M_SCALE*48.25} 0 ${M_SCALE*142.03}" rpy="0 ${M_PI/2.0} 0" />
          <parent link="${prefix}biceps_link" />
-         <child link="${prefix}forearm_link" />
+         <child link="${prefix}forearm_1_link" />
          <axis xyz="0 1 0" />
          <limit lower="-1.571" upper="1.571" effort="6" velocity="1.571" />
@@ -156,5 +143,5 @@
       <joint name="${prefix}joint_4" type="revolute">
          <origin xyz="0 0 ${M_SCALE*142.03}" rpy="0 0 0" />
-         <parent link="${prefix}forearm_link" />
+         <parent link="${prefix}forearm_1_link" />
          <child link="${prefix}wrist_1_link" />
          <axis xyz="0 1 0" />

File: boxbot_description/urdf/widowx_6dof.urdf.xacro (robot description, xacro)
@@ -139,5 +139,5 @@
          <child link="${prefix}arm_base_link"/>
       </joint>
-      <joint name="${prefix}shoulder_joint_1" type="revolute">
+      <joint name="${prefix}joint_1" type="revolute">
          <origin xyz="0 0 0" rpy="0 0 0" />
          <parent link="${prefix}arm_base_link" />
@@ -146,5 +146,5 @@
          <limit lower="-2.617" upper="2.617" effort="6" velocity="0.785" />
       </joint>
-      <joint name="${prefix}shoulder_joint_2" type="revolute">
+      <joint name="${prefix}joint_2" type="revolute">
          <origin xyz="0 0 0" rpy="0 0 ${M_PI}" />
          <parent link="${prefix}shoulder_link" />
@@ -153,5 +153,5 @@
          <limit lower="-1.571" upper="1.571" effort="6" velocity="1.571" />
       </joint>
-      <joint name="${prefix}elbow_joint" type="revolute">
+      <joint name="${prefix}joint_3" type="revolute">
          <origin xyz="-${M_SCALE*48.25} 0 ${M_SCALE*141.8}" rpy="0 ${M_PI/2.0} ${M_PI}" />
          <parent link="${prefix}biceps_link" />
@@ -160,5 +160,5 @@
          <limit lower="-1.571" upper="1.571" effort="6" velocity="1.571" />
       </joint>
-      <joint name="${prefix}wrist_joint_1" type="revolute">
+      <joint name="${prefix}joint_4" type="revolute">
          <origin xyz="0 0 ${M_SCALE*92.8}" rpy="0 0 -${M_PI/2.0}" />
          <parent link="${prefix}forearm_1_link" />
@@ -167,5 +167,5 @@
          <limit lower="-2.617" upper="2.617" effort="2.5" velocity="1.571" />
       </joint>
-      <joint name="${prefix}wrist_joint_2" type="revolute">
+      <joint name="${prefix}joint_5" type="revolute">
          <origin xyz="0 0 0.048" rpy="0 0 ${M_PI/2.0}" />
          <parent link="${prefix}forearm_2_link" />
@@ -174,5 +174,5 @@
          <limit lower="-1.745" upper="1.745" effort="2.5" velocity="1.571" />
       </joint>
-      <joint name="${prefix}wrist_joint_3" type="revolute">
+      <joint name="${prefix}joint_6" type="revolute">
          <origin xyz="0 0 ${M_SCALE*71.5}" rpy="0 0 0" />
          <parent link="${prefix}wrist_1_link" />

File: boxbot_description/urdf/widowx_gripper.xacro (robot description, xacro)
@@ -62,5 +62,5 @@
       </inertial>
    </link>
-   <joint name="${prefix}joint_6" type="fixed">
+   <joint name="${prefix}_rail_joint" type="fixed">
       <origin xyz = "0 0 ${M_SCALE*43}" rpy="0 0 0" />
       <parent link="${prefix}wrist_2_link" />

Commit message: Fix a few minor annoyances

File: boxbot_description/robots/boxbot_5dof.urdf (robot description, URDF)
Before this commit: robot boxbot, 20 links, 19 joints
Joints:
- removed joint left__rail_joint
- removed joint right__rail_joint
- added joint left_rail_joint: type fixed, parent left_wrist_2_link, child left_gripper_rail_link, origin xyz=0 0 0.043 rpy=0 0 0
- added joint right_rail_joint: type fixed, parent right_wrist_2_link, child right_gripper_rail_link, origin xyz=0 0 0.043 rpy=0 0 0

File: boxbot_description/robots/boxbot_6dof.urdf (robot description, URDF)
Before this commit: robot boxbot, 22 links, 21 joints
Joints:
- removed joint left__rail_joint
- removed joint right__rail_joint
- added joint left_rail_joint: type fixed, parent left_wrist_2_link, child left_gripper_rail_link, origin xyz=0 0 0.043 rpy=0 0 0
- added joint right_rail_joint: type fixed, parent right_wrist_2_link, child right_gripper_rail_link, origin xyz=0 0 0.043 rpy=0 0 0

File: boxbot_description/urdf/widowx_gripper.xacro (robot description, xacro)
@@ -62,5 +62,5 @@
       </inertial>
    </link>
-   <joint name="${prefix}_rail_joint" type="fixed">
+   <joint name="${prefix}rail_joint" type="fixed">
       <origin xyz = "0 0 ${M_SCALE*43}" rpy="0 0 0" />
       <parent link="${prefix}wrist_2_link" />
