Commit message: Fix small error in which gripper servo max effort was set to zero.

File: boxbot_description/robots/boxbot_5dof.urdf (robot description, URDF)
Before this commit: robot boxbot, 20 links, 19 joints
Joints:
- joint left_gripper_joint: limit lower=0.002 upper=0.031 effort=0 velocity=0.5 -> lower=0.002 upper=0.031 effort=6 velocity=0.5
- joint left_gripper_prismatic_joint_2: limit lower=0.002 upper=0.031 effort=0 velocity=0.5 -> lower=0.002 upper=0.031 effort=6 velocity=0.5
- joint right_gripper_joint: limit lower=0.002 upper=0.031 effort=0 velocity=0.5 -> lower=0.002 upper=0.031 effort=6 velocity=0.5
- joint right_gripper_prismatic_joint_2: limit lower=0.002 upper=0.031 effort=0 velocity=0.5 -> lower=0.002 upper=0.031 effort=6 velocity=0.5

File: boxbot_description/robots/boxbot_6dof.urdf (robot description, URDF)
Before this commit: robot boxbot, 22 links, 21 joints
Joints:
- joint left_gripper_joint: limit lower=0.002 upper=0.031 effort=0 velocity=0.5 -> lower=0.002 upper=0.031 effort=6 velocity=0.5
- joint left_gripper_prismatic_joint_2: limit lower=0.002 upper=0.031 effort=0 velocity=0.5 -> lower=0.002 upper=0.031 effort=6 velocity=0.5
- joint right_gripper_joint: limit lower=0.002 upper=0.031 effort=0 velocity=0.5 -> lower=0.002 upper=0.031 effort=6 velocity=0.5
- joint right_gripper_prismatic_joint_2: limit lower=0.002 upper=0.031 effort=0 velocity=0.5 -> lower=0.002 upper=0.031 effort=6 velocity=0.5

File: boxbot_description/urdf/widowx_gripper.xacro (robot description, xacro)
@@ -72,5 +72,5 @@
       <child link="${prefix}gripper_1_link" />
       <axis xyz="0 -1 0" />
-      <limit lower="0.002" upper="0.031" effort="0" velocity="0.5" />
+      <limit lower="0.002" upper="0.031" effort="6" velocity="0.5" />
    </joint>
    <joint name="${prefix}gripper_prismatic_joint_2" type="prismatic">
@@ -80,5 +80,5 @@
       <mimic joint="${prefix}gripper_joint" />
       <axis xyz="0 1 0" />
-      <limit lower="0.002" upper="0.031" effort="0" velocity="0.5" />
+      <limit lower="0.002" upper="0.031" effort="6" velocity="0.5" />
    </joint>
 </robot>

Commit message: Update joint names to be more consistent with joint controller names.

File: boxbot_description/robots/boxbot_5dof.urdf (robot description, URDF)
Before this commit: robot boxbot, 20 links, 19 joints
Joints:
- removed joint left_joint_1
- removed joint left_joint_2
- removed joint left_joint_3
- removed joint left_joint_4
- removed joint left_joint_5
- removed joint right_joint_1
- removed joint right_joint_2
- removed joint right_joint_3
- removed joint right_joint_4
- removed joint right_joint_5
- added joint left_elbow_joint: type revolute, parent left_biceps_link, child left_forearm_1_link, origin xyz=0.04825 0 0.14203 rpy=0 1.570795 0, axis 0 1 0, limit lower=-1.571 upper=1.571 effort=6 velocity=1.571
- added joint left_shoulder_1_joint: type revolute, parent left_arm_base_link, child left_shoulder_link, origin xyz=0 0 0 rpy=0 0 0, axis 0 0 1, limit lower=-2.617 upper=2.617 effort=6 velocity=0.785
- added joint left_shoulder_2_joint: type revolute, parent left_shoulder_link, child left_biceps_link, origin xyz=0 0 0 rpy=0 0 0, axis 0 1 0, limit lower=-1.571 upper=1.571 effort=6 velocity=1.571
- added joint left_wrist_1_joint: type revolute, parent left_forearm_1_link, child left_wrist_1_link, origin xyz=0 0 0.14203 rpy=0 0 0, axis 0 1 0, limit lower=-1.745 upper=1.745 effort=6 velocity=1.571
- added joint left_wrist_2_joint: type revolute, parent left_wrist_1_link, child left_wrist_2_link, origin xyz=0 0 0.0715 rpy=0 0 0, axis 0 0 1, limit lower=-2.617 upper=2.617 effort=6 velocity=1.571
- added joint right_elbow_joint: type revolute, parent right_biceps_link, child right_forearm_1_link, origin xyz=0.04825 0 0.14203 rpy=0 1.570795 0, axis 0 1 0, limit lower=-1.571 upper=1.571 effort=6 velocity=1.571
- added joint right_shoulder_1_joint: type revolute, parent right_arm_base_link, child right_shoulder_link, origin xyz=0 0 0 rpy=0 0 0, axis 0 0 1, limit lower=-2.617 upper=2.617 effort=6 velocity=0.785
- added joint right_shoulder_2_joint: type revolute, parent right_shoulder_link, child right_biceps_link, origin xyz=0 0 0 rpy=0 0 0, axis 0 1 0, limit lower=-1.571 upper=1.571 effort=6 velocity=1.571
- added joint right_wrist_1_joint: type revolute, parent right_forearm_1_link, child right_wrist_1_link, origin xyz=0 0 0.14203 rpy=0 0 0, axis 0 1 0, limit lower=-1.745 upper=1.745 effort=6 velocity=1.571
- added joint right_wrist_2_joint: type revolute, parent right_wrist_1_link, child right_wrist_2_link, origin xyz=0 0 0.0715 rpy=0 0 0, axis 0 0 1, limit lower=-2.617 upper=2.617 effort=6 velocity=1.571

File: boxbot_description/robots/boxbot_6dof.urdf (robot description, URDF)
Before this commit: robot boxbot, 22 links, 21 joints
Joints:
- removed joint left_joint_1
- removed joint left_joint_2
- removed joint left_joint_3
- removed joint left_joint_4
- removed joint left_joint_5
- removed joint left_joint_6
- removed joint right_joint_1
- removed joint right_joint_2
- removed joint right_joint_3
- removed joint right_joint_4
- removed joint right_joint_5
- removed joint right_joint_6
- added joint left_elbow_joint: type revolute, parent left_biceps_link, child left_forearm_1_link, origin xyz=-0.04825 0 0.1418 rpy=0 1.570795 3.14159, axis 0 -1 0, limit lower=-1.571 upper=1.571 effort=6 velocity=1.571
- added joint left_shoulder_1_joint: type revolute, parent left_arm_base_link, child left_shoulder_link, origin xyz=0 0 0 rpy=0 0 0, axis 0 0 1, limit lower=-2.617 upper=2.617 effort=6 velocity=0.785
- added joint left_shoulder_2_joint: type revolute, parent left_shoulder_link, child left_biceps_link, origin xyz=0 0 0 rpy=0 0 3.14159, axis 0 1 0, limit lower=-1.571 upper=1.571 effort=6 velocity=1.571
- added joint left_wrist_1_joint: type revolute, parent left_forearm_1_link, child left_forearm_2_link, origin xyz=0 0 0.0928 rpy=0 0 -1.570795, axis 0 0 1, limit lower=-2.617 upper=2.617 effort=2.5 velocity=1.571
- added joint left_wrist_2_joint: type revolute, parent left_forearm_2_link, child left_wrist_1_link, origin xyz=0 0 0.048 rpy=0 0 1.570795, axis 0 1 0, limit lower=-1.745 upper=1.745 effort=2.5 velocity=1.571
- added joint left_wrist_3_joint: type revolute, parent left_wrist_1_link, child left_wrist_2_link, origin xyz=0 0 0.0715 rpy=0 0 0, axis 0 0 1, limit lower=-2.617 upper=2.617 effort=1.5 velocity=1.571
- added joint right_elbow_joint: type revolute, parent right_biceps_link, child right_forearm_1_link, origin xyz=-0.04825 0 0.1418 rpy=0 1.570795 3.14159, axis 0 -1 0, limit lower=-1.571 upper=1.571 effort=6 velocity=1.571
- added joint right_shoulder_1_joint: type revolute, parent right_arm_base_link, child right_shoulder_link, origin xyz=0 0 0 rpy=0 0 0, axis 0 0 1, limit lower=-2.617 upper=2.617 effort=6 velocity=0.785
- added joint right_shoulder_2_joint: type revolute, parent right_shoulder_link, child right_biceps_link, origin xyz=0 0 0 rpy=0 0 3.14159, axis 0 1 0, limit lower=-1.571 upper=1.571 effort=6 velocity=1.571
- added joint right_wrist_1_joint: type revolute, parent right_forearm_1_link, child right_forearm_2_link, origin xyz=0 0 0.0928 rpy=0 0 -1.570795, axis 0 0 1, limit lower=-2.617 upper=2.617 effort=2.5 velocity=1.571
- added joint right_wrist_2_joint: type revolute, parent right_forearm_2_link, child right_wrist_1_link, origin xyz=0 0 0.048 rpy=0 0 1.570795, axis 0 1 0, limit lower=-1.745 upper=1.745 effort=2.5 velocity=1.571
- added joint right_wrist_3_joint: type revolute, parent right_wrist_1_link, child right_wrist_2_link, origin xyz=0 0 0.0715 rpy=0 0 0, axis 0 0 1, limit lower=-2.617 upper=2.617 effort=1.5 velocity=1.571

File: boxbot_description/urdf/servos.urdf.xacro (robot description, xacro)
@@ -12,5 +12,5 @@
     <transmission name="ltran1">
       <type>transmission_interface/SimpleTransmission</type>
-      <joint name="left_joint_1">
+      <joint name="left_shoulder_1_joint">
         <hardwareInterface>hardware_interface/PositionJointInterface</hardwareInterface>
       </joint>
@@ -22,5 +22,5 @@
     <transmission name="ltran2">
       <type>transmission_interface/SimpleTransmission</type>
-      <joint name="left_joint_2">
+      <joint name="left_shoulder_2_joint">
         <hardwareInterface>hardware_interface/PositionJointInterface</hardwareInterface>
       </joint>
@@ -32,5 +32,5 @@
     <transmission name="ltran3">
       <type>transmission_interface/SimpleTransmission</type>
-      <joint name="left_joint_3">
+      <joint name="left_elbow_joint">
         <hardwareInterface>hardware_interface/PositionJointInterface</hardwareInterface>
       </joint>
@@ -42,5 +42,5 @@
     <transmission name="ltran4">
       <type>transmission_interface/SimpleTransmission</type>
-      <joint name="left_joint_4">
+      <joint name="left_wrist_1_joint">
         <hardwareInterface>hardware_interface/PositionJointInterface</hardwareInterface>
       </joint>
@@ -52,5 +52,5 @@
     <transmission name="ltran5">
       <type>transmission_interface/SimpleTransmission</type>
-      <joint name="left_joint_5">
+      <joint name="left_wrist_2_joint">
         <hardwareInterface>hardware_interface/PositionJointInterface</hardwareInterface>
       </joint>
@@ -63,5 +63,5 @@
       <transmission name="ltran6">
         <type>transmission_interface/SimpleTransmission</type>
-        <joint name="left_joint_6">
+        <joint name="left_wrist_3_joint">
           <hardwareInterface>hardware_interface/PositionJointInterface</hardwareInterface>
         </joint>
@@ -95,5 +95,5 @@
     <transmission name="rtran1">
       <type>transmission_interface/SimpleTransmission</type>
-      <joint name="right_joint_1">
+      <joint name="right_shoulder_1_joint">
         <hardwareInterface>hardware_interface/PositionJointInterface</hardwareInterface>
       </joint>
@@ -105,5 +105,5 @@
     <transmission name="rtran2">
       <type>transmission_interface/SimpleTransmission</type>
-      <joint name="right_joint_2">
+      <joint name="right_shoulder_2_joint">
         <hardwareInterface>hardware_interface/PositionJointInterface</hardwareInterface>
       </joint>
@@ -115,5 +115,5 @@
     <transmission name="rtran3">
       <type>transmission_interface/SimpleTransmission</type>
-      <joint name="right_joint_3">
+      <joint name="right_elbow_joint">
         <hardwareInterface>hardware_interface/PositionJointInterface</hardwareInterface>
       </joint>
@@ -125,5 +125,5 @@
     <transmission name="rtran4">
       <type>transmission_interface/SimpleTransmission</type>
-      <joint name="right_joint_4">
+      <joint name="right_wrist_1_joint">
         <hardwareInterface>hardware_interface/PositionJointInterface</hardwareInterface>
       </joint>
@@ -135,5 +135,5 @@
     <transmission name="rtran5">
       <type>transmission_interface/SimpleTransmission</type>
-      <joint name="right_joint_5">
+      <joint name="right_wrist_2_joint">
         <hardwareInterface>hardware_interface/PositionJointInterface</hardwareInterface>
       </joint>
@@ -146,5 +146,5 @@
       <transmission name="rtran6">
         <type>transmission_interface/SimpleTransmission</type>
-        <joint name="right_joint_6">
+        <joint name="right_wrist_3_joint">
           <hardwareInterface>hardware_interface/PositionJointInterface</hardwareInterface>
         </joint>

File: boxbot_description/urdf/widowx.urdf.xacro (robot description, xacro)
@@ -119,5 +119,5 @@
          <child link="${prefix}arm_base_link"/>
       </joint>
-      <joint name="${prefix}joint_1" type="revolute">
+      <joint name="${prefix}shoulder_1_joint" type="revolute">
          <origin xyz="0 0 0" rpy="0 0 0" />
          <parent link="${prefix}arm_base_link" />
@@ -126,5 +126,5 @@
          <limit lower="-2.617" upper="2.617" effort="6" velocity="0.785" />
       </joint>
-      <joint name="${prefix}joint_2" type="revolute">
+      <joint name="${prefix}shoulder_2_joint" type="revolute">
          <!--origin xyz="0.04825 0 0.14203" rpy="0 0 0" /-->
          <origin xyz="0 0 0" rpy="0 0 0" />
@@ -134,5 +134,5 @@
          <limit lower="-1.571" upper="1.571" effort="6" velocity="1.571" />
       </joint>
-      <joint name="${prefix}joint_3" type="revolute">
+      <joint name="${prefix}elbow_joint" type="revolute">
          <origin xyz="${M_SCALE*48.25} 0 ${M_SCALE*142.03}" rpy="0 ${M_PI/2.0} 0" />
          <parent link="${prefix}biceps_link" />
@@ -141,5 +141,5 @@
          <limit lower="-1.571" upper="1.571" effort="6" velocity="1.571" />
       </joint>
-      <joint name="${prefix}joint_4" type="revolute">
+      <joint name="${prefix}wrist_1_joint" type="revolute">
          <origin xyz="0 0 ${M_SCALE*142.03}" rpy="0 0 0" />
          <parent link="${prefix}forearm_1_link" />
@@ -148,5 +148,5 @@
          <limit lower="-1.745" upper="1.745" effort="6" velocity="1.571" />
       </joint>
-      <joint name="${prefix}joint_5" type="revolute">
+      <joint name="${prefix}wrist_2_joint" type="revolute">
          <origin xyz="0 0 ${M_SCALE*71.5}" rpy="0 0 0" />
          <parent link="${prefix}wrist_1_link" />

File: boxbot_description/urdf/widowx_6dof.urdf.xacro (robot description, xacro)
@@ -139,5 +139,5 @@
          <child link="${prefix}arm_base_link"/>
       </joint>
-      <joint name="${prefix}joint_1" type="revolute">
+      <joint name="${prefix}shoulder_1_joint" type="revolute">
          <origin xyz="0 0 0" rpy="0 0 0" />
          <parent link="${prefix}arm_base_link" />
@@ -146,5 +146,5 @@
          <limit lower="-2.617" upper="2.617" effort="6" velocity="0.785" />
       </joint>
-      <joint name="${prefix}joint_2" type="revolute">
+      <joint name="${prefix}shoulder_2_joint" type="revolute">
          <origin xyz="0 0 0" rpy="0 0 ${M_PI}" />
          <parent link="${prefix}shoulder_link" />
@@ -153,5 +153,5 @@
          <limit lower="-1.571" upper="1.571" effort="6" velocity="1.571" />
       </joint>
-      <joint name="${prefix}joint_3" type="revolute">
+      <joint name="${prefix}elbow_joint" type="revolute">
          <origin xyz="-${M_SCALE*48.25} 0 ${M_SCALE*141.8}" rpy="0 ${M_PI/2.0} ${M_PI}" />
          <parent link="${prefix}biceps_link" />
@@ -160,5 +160,5 @@
          <limit lower="-1.571" upper="1.571" effort="6" velocity="1.571" />
       </joint>
-      <joint name="${prefix}joint_4" type="revolute">
+      <joint name="${prefix}wrist_1_joint" type="revolute">
          <origin xyz="0 0 ${M_SCALE*92.8}" rpy="0 0 -${M_PI/2.0}" />
          <parent link="${prefix}forearm_1_link" />
@@ -167,5 +167,5 @@
          <limit lower="-2.617" upper="2.617" effort="2.5" velocity="1.571" />
       </joint>
-      <joint name="${prefix}joint_5" type="revolute">
+      <joint name="${prefix}wrist_2_joint" type="revolute">
          <origin xyz="0 0 0.048" rpy="0 0 ${M_PI/2.0}" />
          <parent link="${prefix}forearm_2_link" />
@@ -174,5 +174,5 @@
          <limit lower="-1.745" upper="1.745" effort="2.5" velocity="1.571" />
       </joint>
-      <joint name="${prefix}joint_6" type="revolute">
+      <joint name="${prefix}wrist_3_joint" type="revolute">
          <origin xyz="0 0 ${M_SCALE*71.5}" rpy="0 0 0" />
          <parent link="${prefix}wrist_1_link" />
