Commit message: Add gazebo plugin cameras to model

File: boxbot_description/robots/boxbot_5dof.urdf (robot description, URDF)
Before this commit: robot boxbot, 20 links, 19 joints
Links:
- added link left_camera_link, mass 0.001; collision cylinder length=0.003 radius=0.014; visual cylinder length=0.003 radius=0.014
- added link neck_base_link, mass 0.001; collision cylinder length=0.02 radius=0.02; visual cylinder length=0.02 radius=0.02
- added link pan_link, mass 0.001; collision box size=0.039 0.09 0.04; visual box size=0.039 0.09 0.04
- added link right_camera_link, mass 0.001; collision cylinder length=0.003 radius=0.014; visual cylinder length=0.003 radius=0.014
- added link tilt_link, mass 0.001; collision box size=0.02 0.1 0.005; visual box size=0.02 0.1 0.005
Joints:
- added joint left_camera_joint: type fixed, parent tilt_link, child left_camera_link, origin xyz=0.023 0.045 0.005 rpy=0 -1.5707963267948966 0
- added joint neck_base_joint: type fixed, parent torso, child neck_base_link, origin xyz=0 0 0.342 rpy=0 0 0
- added joint pan_joint: type revolute, parent neck_base_link, child pan_link, origin xyz=0 0 0.012 rpy=0 0 0, axis 0 0 1, limit lower=-3.14 upper=3.14 effort=3 velocity=3.141592653589793
- added joint right_camera_joint: type fixed, parent tilt_link, child right_camera_link, origin xyz=0.023 -0.045 0.005 rpy=0 -1.5707963267948966 0
- added joint tilt_joint: type revolute, parent pan_link, child tilt_link, origin xyz=0.055 0 0.025 rpy=0 0 0, axis 0 1 0, limit lower=-1.5707963267948966 upper=0.50 effort=3 velocity=3.141592653589793
- joint left_arm_base_joint: origin xyz=0 0.099613 0.24953 rpy=-1.570795 0 0 -> xyz=0 0.09961300000000001 0.24953 rpy=-1.570795 0 0
- joint left_elbow_joint: origin xyz=0.04825 0 0.14203 rpy=0 1.570795 0 -> xyz=0.04825 0 0.14203000000000002 rpy=0 1.570795 0
- joint left_rail_joint: origin xyz=0 0 0.043 rpy=0 0 0 -> xyz=0 0 0.043000000000000003 rpy=0 0 0
- joint left_wrist_1_joint: origin xyz=0 0 0.14203 rpy=0 0 0 -> xyz=0 0 0.14203000000000002 rpy=0 0 0
- joint left_wrist_2_joint: origin xyz=0 0 0.0715 rpy=0 0 0 -> xyz=0 0 0.07150000000000001 rpy=0 0 0
- joint right_arm_base_joint: origin xyz=0 -0.099613 0.24953 rpy=1.570795 0 0 -> xyz=0 -0.09961300000000001 0.24953 rpy=1.570795 0 0
- joint right_elbow_joint: origin xyz=0.04825 0 0.14203 rpy=0 1.570795 0 -> xyz=0.04825 0 0.14203000000000002 rpy=0 1.570795 0
- joint right_rail_joint: origin xyz=0 0 0.043 rpy=0 0 0 -> xyz=0 0 0.043000000000000003 rpy=0 0 0
- joint right_wrist_1_joint: origin xyz=0 0 0.14203 rpy=0 0 0 -> xyz=0 0 0.14203000000000002 rpy=0 0 0
- joint right_wrist_2_joint: origin xyz=0 0 0.0715 rpy=0 0 0 -> xyz=0 0 0.07150000000000001 rpy=0 0 0

File: boxbot_description/robots/boxbot_5dof.urdf.xacro (robot description, xacro)
@@ -38,7 +38,12 @@
     <origin xyz="0 -${M_SCALE*99.613} ${M_SCALE*249.53}" rpy="${M_PI/2.0} 0 0"/>
   </xacro:widowx_arm>
+  <xacro:include filename="$(find boxbot_description)/urdf/head.urdf.xacro"/>
+  <xacro:boxbot_head parent="torso">
+    <origin xyz="0 0 ${M_SCALE*342.0}" rpy="0 0 0"/>
+  </xacro:boxbot_head>
+  <xacro:include filename="$(find boxbot_description)/urdf/sensors.gazebo"/>
   <xacro:include filename="$(find boxbot_description)/urdf/servos.urdf.xacro"/>
-  <xacro:ros_control_widowx six_dof="false"/>
+  <xacro:ros_control_widowx six_dof="true" head="true"/>
   <xacro:include filename="$(find boxbot_description)/urdf/materials.gazebo"/>
-  <xacro:gazebo_widowx six_dof="false"/>
+  <xacro:gazebo_widowx six_dof="true" head="true"/>
 </robot>

File: boxbot_description/robots/boxbot_6dof.urdf (robot description, URDF)
Before this commit: robot boxbot, 22 links, 21 joints
Links:
- added link left_camera_link, mass 0.001; collision cylinder length=0.003 radius=0.014; visual cylinder length=0.003 radius=0.014
- added link neck_base_link, mass 0.001; collision cylinder length=0.02 radius=0.02; visual cylinder length=0.02 radius=0.02
- added link pan_link, mass 0.001; collision box size=0.039 0.09 0.04; visual box size=0.039 0.09 0.04
- added link right_camera_link, mass 0.001; collision cylinder length=0.003 radius=0.014; visual cylinder length=0.003 radius=0.014
- added link tilt_link, mass 0.001; collision box size=0.02 0.1 0.005; visual box size=0.02 0.1 0.005
Joints:
- added joint left_camera_joint: type fixed, parent tilt_link, child left_camera_link, origin xyz=0.023 0.045 0.005 rpy=0 -1.5707963267948966 0
- added joint neck_base_joint: type fixed, parent torso, child neck_base_link, origin xyz=0 0 0.342 rpy=0 0 0
- added joint pan_joint: type revolute, parent neck_base_link, child pan_link, origin xyz=0 0 0.012 rpy=0 0 0, axis 0 0 1, limit lower=-3.14 upper=3.14 effort=3 velocity=3.141592653589793
- added joint right_camera_joint: type fixed, parent tilt_link, child right_camera_link, origin xyz=0.023 -0.045 0.005 rpy=0 -1.5707963267948966 0
- added joint tilt_joint: type revolute, parent pan_link, child tilt_link, origin xyz=0.055 0 0.025 rpy=0 0 0, axis 0 1 0, limit lower=-1.5707963267948966 upper=0.50 effort=3 velocity=3.141592653589793
- joint left_arm_base_joint: origin xyz=0 0.099613 0.24953 rpy=-1.570795 0 0 -> xyz=0 0.09961300000000001 0.24953 rpy=-1.570795 0 0
- joint left_rail_joint: origin xyz=0 0 0.043 rpy=0 0 0 -> xyz=0 0 0.043000000000000003 rpy=0 0 0
- joint left_wrist_3_joint: origin xyz=0 0 0.0715 rpy=0 0 0 -> xyz=0 0 0.07150000000000001 rpy=0 0 0
- joint right_arm_base_joint: origin xyz=0 -0.099613 0.24953 rpy=1.570795 0 0 -> xyz=0 -0.09961300000000001 0.24953 rpy=1.570795 0 0
- joint right_rail_joint: origin xyz=0 0 0.043 rpy=0 0 0 -> xyz=0 0 0.043000000000000003 rpy=0 0 0
- joint right_wrist_3_joint: origin xyz=0 0 0.0715 rpy=0 0 0 -> xyz=0 0 0.07150000000000001 rpy=0 0 0

File: boxbot_description/robots/boxbot_6dof.urdf.xacro (robot description, xacro)
@@ -38,7 +38,12 @@
     <origin xyz="0 -${M_SCALE*99.613} ${M_SCALE*249.53}" rpy="${M_PI/2.0} 0 0"/>
   </xacro:widowx_arm>
+  <xacro:include filename="$(find boxbot_description)/urdf/head.urdf.xacro"/>
+  <xacro:boxbot_head parent="torso">
+    <origin xyz="0 0 ${M_SCALE*342.0}" rpy="0 0 0"/>
+  </xacro:boxbot_head>
+  <xacro:include filename="$(find boxbot_description)/urdf/sensors.gazebo"/>
   <xacro:include filename="$(find boxbot_description)/urdf/servos.urdf.xacro"/>
-  <xacro:ros_control_widowx six_dof="true"/>
+  <xacro:ros_control_widowx six_dof="true" head="true"/>
   <xacro:include filename="$(find boxbot_description)/urdf/materials.gazebo"/>
-  <xacro:gazebo_widowx six_dof="true"/>
+  <xacro:gazebo_widowx six_dof="true" head="true"/>
 </robot>

File: boxbot_description/urdf/servos.urdf.xacro (robot description, xacro)
@@ -1,5 +1,5 @@
 <?xml version="1.0"?>
 <robot xmlns:xacro="http://ros.org/wiki/xacro">
-  <xacro:macro name="ros_control_widowx" params="six_dof">
+  <xacro:macro name="ros_control_widowx" params="six_dof head">
     <!--gazebo ros control-->
     <gazebo>
@@ -175,4 +175,29 @@
       </actuator>
     </transmission>
+    <!-- head -->
+    <xacro:if value="${head}">
+      <transmission name="htran1">
+        <type>transmission_interface/SimpleTransmission</type>
+        <joint name="pan_joint">
+          <hardwareInterface>hardware_interface/PositionJointInterface</hardwareInterface>
+        </joint>
+        <actuator name="head_motor1">
+          <hardwareInterface>hardware_interface/PositionJointInterface</hardwareInterface>
+          <mechanicalReduction>1</mechanicalReduction>
+        </actuator>
+      </transmission>
+    </xacro:if>
+    <xacro:if value="${head}">
+      <transmission name="htran2">
+        <type>transmission_interface/SimpleTransmission</type>
+        <joint name="tilt_joint">
+          <hardwareInterface>hardware_interface/PositionJointInterface</hardwareInterface>
+        </joint>
+        <actuator name="head_motor2">
+          <hardwareInterface>hardware_interface/PositionJointInterface</hardwareInterface>
+          <mechanicalReduction>1</mechanicalReduction>
+        </actuator>
+      </transmission>
+    </xacro:if>
   </xacro:macro>
 </robot>
