Commit message: Reorganize and refactor main URDF elements

File: boxbot_description/robots/boxbot_5dof.urdf.xacro (robot description, xacro)
@@ -2,5 +2,5 @@
 <robot name="boxbot" xmlns:xacro="http://ros.org/wiki/xacro">
   <xacro:property name="M_SCALE" value="0.001"/>
-  <xacro:include filename="$(find boxbot_description)/urdf/common_materials.xacro" />
+  <xacro:include filename="$(find boxbot_description)/xacro/common_materials.xacro" />
   <link name="world"/>
   <link name="torso">
@@ -30,20 +30,20 @@
     <child link="torso"/>
   </joint>
-  <xacro:include filename="$(find boxbot_description)/urdf/widowx.urdf.xacro"/>
-  <xacro:widowx_arm parent="torso" prefix="left_">
+  <xacro:include filename="$(find boxbot_description)/xacro/widowx.urdf.xacro"/>
+  <xacro:widowx_arm parent="torso" prefix="left_" six_dof="false">
     <origin xyz="0 ${M_SCALE*99.613} ${M_SCALE*249.53}" rpy="-${M_PI/2.0} 0 0" />
   </xacro:widowx_arm>
-  <xacro:include filename="$(find boxbot_description)/urdf/widowx.urdf.xacro"/>
-  <xacro:widowx_arm parent="torso" prefix="right_">
+  <xacro:include filename="$(find boxbot_description)/xacro/widowx.urdf.xacro"/>
+  <xacro:widowx_arm parent="torso" prefix="right_" six_dof="false">
     <origin xyz="0 -${M_SCALE*99.613} ${M_SCALE*249.53}" rpy="${M_PI/2.0} 0 0"/>
   </xacro:widowx_arm>
-  <xacro:include filename="$(find boxbot_description)/urdf/head.urdf.xacro"/>
+  <xacro:include filename="$(find boxbot_description)/xacro/head.urdf.xacro"/>
   <xacro:boxbot_head parent="torso">
     <origin xyz="0 0 ${M_SCALE*342.0}" rpy="0 0 0"/>
   </xacro:boxbot_head>
-  <xacro:include filename="$(find boxbot_description)/urdf/sensors.gazebo"/>
-  <xacro:include filename="$(find boxbot_description)/urdf/servos.urdf.xacro"/>
+  <!--xacro:include filename="$(find boxbot_description)/xacro/sensors.gazebo"/>
+  <xacro:include filename="$(find boxbot_description)/xacro/servos.urdf.xacro"/>
   <xacro:ros_control_widowx six_dof="true" head="true"/>
-  <xacro:include filename="$(find boxbot_description)/urdf/materials.gazebo"/>
-  <xacro:gazebo_widowx six_dof="true" head="true"/>
+  <xacro:include filename="$(find boxbot_description)/xacro/materials.gazebo"/>
+  <xacro:gazebo_widowx six_dof="true" head="true"/-->
 </robot>

File: boxbot_description/robots/boxbot_6dof.urdf.xacro (robot description, xacro)
@@ -2,5 +2,5 @@
 <robot name="boxbot" xmlns:xacro="http://ros.org/wiki/xacro">
   <xacro:property name="M_SCALE" value="0.001"/>
-  <xacro:include filename="$(find boxbot_description)/urdf/common_materials.xacro" />
+  <xacro:include filename="$(find boxbot_description)/xacro/common_materials.xacro" />
   <link name="world"/>
   <link name="torso">
@@ -30,20 +30,20 @@
     <child link="torso"/>
   </joint>
-  <xacro:include filename="$(find boxbot_description)/urdf/widowx_6dof.urdf.xacro"/>
-  <xacro:widowx_arm parent="torso" prefix="left_">
+  <xacro:include filename="$(find boxbot_description)/xacro/widowx.urdf.xacro"/>
+  <xacro:widowx_arm parent="torso" prefix="left_" six_dof="true">
     <origin xyz="0 ${M_SCALE*99.613} ${M_SCALE*249.53}" rpy="-${M_PI/2.0} 0 0" />
   </xacro:widowx_arm>
-  <xacro:include filename="$(find boxbot_description)/urdf/widowx_6dof.urdf.xacro"/>
-  <xacro:widowx_arm parent="torso" prefix="right_">
+  <xacro:include filename="$(find boxbot_description)/xacro/widowx.urdf.xacro"/>
+  <xacro:widowx_arm parent="torso" prefix="right_" six_dof="true">
     <origin xyz="0 -${M_SCALE*99.613} ${M_SCALE*249.53}" rpy="${M_PI/2.0} 0 0"/>
   </xacro:widowx_arm>
-  <xacro:include filename="$(find boxbot_description)/urdf/head.urdf.xacro"/>
+  <xacro:include filename="$(find boxbot_description)/xacro/head.urdf.xacro"/>
   <xacro:boxbot_head parent="torso">
     <origin xyz="0 0 ${M_SCALE*342.0}" rpy="0 0 0"/>
   </xacro:boxbot_head>
-  <xacro:include filename="$(find boxbot_description)/urdf/sensors.gazebo"/>
-  <xacro:include filename="$(find boxbot_description)/urdf/servos.urdf.xacro"/>
+  <!--xacro:include filename="$(find boxbot_description)/xacro/sensors.gazebo"/>
+  <xacro:include filename="$(find boxbot_description)/xacro/servos.urdf.xacro"/>
   <xacro:ros_control_widowx six_dof="true" head="true"/>
-  <xacro:include filename="$(find boxbot_description)/urdf/materials.gazebo"/>
-  <xacro:gazebo_widowx six_dof="true" head="true"/>
+  <xacro:include filename="$(find boxbot_description)/xacro/materials.gazebo"/>
+  <xacro:gazebo_widowx six_dof="true" head="true"/-->
 </robot>

File: boxbot_description/xacro/common_materials.xacro (robot description, xacro)
@@ -1,5 +1,5 @@
 <?xml version="1.0"?>
 <robot xmlns:xacro="http://ros.org/wiki/xacro">
-	<xacro:include filename="$(find boxbot_description)/urdf/common_colours.xacro"/>
+	<xacro:include filename="$(find boxbot_description)/xacro/common_colours.xacro"/>
 	<xacro:macro name="material_yellow">
 		<material name="">

File: boxbot_description/xacro/head.urdf.xacro (robot description, xacro)
@@ -1,5 +1,5 @@
 <?xml version="1.0" encoding="UTF-8"?>
 <robot xmlns:xacro="http://ros.org/wiki/xacro">
-  <xacro:include filename="$(find boxbot_description)/urdf/common_materials.xacro" />
+  <xacro:include filename="$(find boxbot_description)/xacro/common_materials.xacro" />
   <xacro:macro name="boxbot_head" params="parent *origin">
     <!-- links -->
@@ -33,5 +33,5 @@
       </visual>
       <collision>
-        <origin rpy="0 0 ${pi/2}" xyz="0 0 -0.0022"/>
+        <origin rpy="0 0 ${pi/2}" xyz="0.02 0 0.017"/>
         <geometry>
           <box size="0.039 0.09 0.04"/>
@@ -134,4 +134,4 @@
       <child link="right_camera_link"/>
     </joint>
- </xacro:macro>
+  </xacro:macro>
 </robot>

Commit message: Update URDF ros control interfaces for ros2 control

File: boxbot_description/robots/boxbot_5dof.urdf.xacro (robot description, xacro)
@@ -42,6 +42,15 @@
     <origin xyz="0 0 ${M_SCALE*342.0}" rpy="0 0 0"/>
   </xacro:boxbot_head>
-  <!--xacro:include filename="$(find boxbot_description)/xacro/sensors.gazebo"/>
-  <xacro:include filename="$(find boxbot_description)/xacro/servos.urdf.xacro"/>
+  <!-- ros2_control -->
+  <xacro:include filename="$(find boxbot_description)/xacro/boxbot.ros2_control.xacro"/>
+  <xacro:widowx_ros2_control name="left_arm_interface" prefix="left_" six_dof="false" use_gazebo="true"/>
+  <xacro:widowx_ros2_control name="right_arm_interface" prefix="right_" six_dof="false" use_gazebo="true"/>
+  <xacro:pan_tilt_head name="head_interface" use_gazebo="true"/>
+  <gazebo>
+    <plugin filename="libgz_ros2_control-system.so" name="gz_ros2_control::GazeboSimROS2ControlPlugin">
+      <parameters>$(find boxbot_control)/config/boxbot_control.yaml</parameters>
+    </plugin>
+  </gazebo>
+  <!--xacro:include filename="$(find boxbot_description)/xacro/servos.urdf.xacro"/>
   <xacro:ros_control_widowx six_dof="true" head="true"/>
   <xacro:include filename="$(find boxbot_description)/xacro/materials.gazebo"/>

File: boxbot_description/robots/boxbot_6dof.urdf.xacro (robot description, xacro)
@@ -42,6 +42,15 @@
     <origin xyz="0 0 ${M_SCALE*342.0}" rpy="0 0 0"/>
   </xacro:boxbot_head>
-  <!--xacro:include filename="$(find boxbot_description)/xacro/sensors.gazebo"/>
-  <xacro:include filename="$(find boxbot_description)/xacro/servos.urdf.xacro"/>
+  <!-- ros2_control -->
+  <xacro:include filename="$(find boxbot_description)/xacro/boxbot.ros2_control.xacro"/>
+  <xacro:widowx_ros2_control name="left_arm_interface" prefix="left_" six_dof="true" use_gazebo="true"/>
+  <xacro:widowx_ros2_control name="right_arm_interface" prefix="right_" six_dof="true" use_gazebo="true"/>
+  <xacro:pan_tilt_head name="head_interface" use_gazebo="true"/>
+  <gazebo>
+    <plugin filename="libgz_ros2_control-system.so" name="gz_ros2_control::GazeboSimROS2ControlPlugin">
+      <parameters>$(find boxbot_control)/config/boxbot_control.yaml</parameters>
+    </plugin>
+  </gazebo>
+  <!--xacro:include filename="$(find boxbot_description)/xacro/servos.urdf.xacro"/>
   <xacro:ros_control_widowx six_dof="true" head="true"/>
   <xacro:include filename="$(find boxbot_description)/xacro/materials.gazebo"/>

File: boxbot_description/xacro/head.urdf.xacro (robot description, xacro)
@@ -53,5 +53,5 @@
       </visual>
       <collision>
-        <origin rpy="0 0 0" xyz="0 0 0"/>
+        <origin rpy="0 ${radians(-90)} 0" xyz="0.02 0 0"/>
         <geometry>
           <box size="0.02 0.1 0.005"/>
@@ -134,4 +134,12 @@
       <child link="right_camera_link"/>
     </joint>
+    <!--xacro:include filename="$(find boxbot_description)/xacro/camera.xacro"/>
+    <xacro:rgb_camera parent="tilt_link" prefix="left_">
+      <origin rpy="0 ${radians(-90)} 0" xyz="0.023 0.045 0.005"/>
+    </xacro:rgb_camera>
+    <xacro:include filename="$(find boxbot_description)/xacro/camera.xacro"/>
+    <xacro:rgb_camera parent="tilt_link" prefix="right_">
+      <origin rpy="0 ${radians(-90)} 0" xyz="0.023 -0.045 0.005"/>
+    </xacro:rgb_camera-->
   </xacro:macro>
 </robot>

File: boxbot_description/xacro/widowx_gripper.xacro (robot description, xacro)
@@ -80,5 +80,5 @@
     <parent link="${prefix}gripper_rail_link" />
     <child link="${prefix}gripper_2_link" />
-    <mimic joint="${prefix}gripper_joint" />
+    <!--mimic joint="${prefix}gripper_joint" /-->
     <axis xyz="0 1 0" />
     <limit lower="0.002" upper="0.031" effort="6" velocity="0.5" />

Commit message: Switch to Bullet physics engine to fix gripper mimic

File: boxbot_description/robots/boxbot_5dof.urdf.xacro (robot description, xacro)
@@ -46,5 +46,5 @@
   <xacro:widowx_ros2_control name="left_arm_interface" prefix="left_" six_dof="false" use_gazebo="true"/>
   <xacro:widowx_ros2_control name="right_arm_interface" prefix="right_" six_dof="false" use_gazebo="true"/>
-  <xacro:pan_tilt_head name="head_interface" use_gazebo="true"/>
+  <xacro:head_ros2_control name="head_interface" use_gazebo="true"/>
   <gazebo>
     <plugin filename="libgz_ros2_control-system.so" name="gz_ros2_control::GazeboSimROS2ControlPlugin">

File: boxbot_description/robots/boxbot_6dof.urdf.xacro (robot description, xacro)
@@ -46,5 +46,5 @@
   <xacro:widowx_ros2_control name="left_arm_interface" prefix="left_" six_dof="true" use_gazebo="true"/>
   <xacro:widowx_ros2_control name="right_arm_interface" prefix="right_" six_dof="true" use_gazebo="true"/>
-  <xacro:pan_tilt_head name="head_interface" use_gazebo="true"/>
+  <xacro:head_ros2_control name="head_interface" use_gazebo="true"/>
   <gazebo>
     <plugin filename="libgz_ros2_control-system.so" name="gz_ros2_control::GazeboSimROS2ControlPlugin">
@@ -52,7 +52,5 @@
     </plugin>
   </gazebo>
-  <!--xacro:include filename="$(find boxbot_description)/xacro/servos.urdf.xacro"/>
-  <xacro:ros_control_widowx six_dof="true" head="true"/>
-  <xacro:include filename="$(find boxbot_description)/xacro/materials.gazebo"/>
+  <!--xacro:include filename="$(find boxbot_description)/xacro/materials.gazebo"/>
   <xacro:gazebo_widowx six_dof="true" head="true"/-->
 </robot>

File: boxbot_description/xacro/boxbot.ros2_control.xacro (robot description, xacro)
@@ -78,14 +78,7 @@
         <state_interface name="position"/>
       </joint>
-      <joint name="${prefix}gripper_prismatic_joint_2">
-        <command_interface name="position">
-          <param name="min">0.002</param>
-          <param name="max">0.031</param>
-        </command_interface>
-        <state_interface name="position"/>
-      </joint>
     </ros2_control>
   </xacro:macro>
-  <xacro:macro name="pan_tilt_head"  params="name use_gazebo">
+  <xacro:macro name="head_ros2_control"  params="name use_gazebo">
     <ros2_control name="${name}" type="system">
       <hardware>

File: boxbot_description/xacro/widowx_gripper.xacro (robot description, xacro)
@@ -80,5 +80,5 @@
     <parent link="${prefix}gripper_rail_link" />
     <child link="${prefix}gripper_2_link" />
-    <!--mimic joint="${prefix}gripper_joint" /-->
+    <mimic joint="${prefix}gripper_joint" multiplier="1.0" offset="0"/>
     <axis xyz="0 1 0" />
     <limit lower="0.002" upper="0.031" effort="6" velocity="0.5" />

Commit message: Update camera sensors for Gazebo Harmonic

File: boxbot_description/robots/boxbot_5dof.urdf.xacro (robot description, xacro)
@@ -52,7 +52,5 @@
     </plugin>
   </gazebo>
-  <!--xacro:include filename="$(find boxbot_description)/xacro/servos.urdf.xacro"/>
-  <xacro:ros_control_widowx six_dof="true" head="true"/>
-  <xacro:include filename="$(find boxbot_description)/xacro/materials.gazebo"/>
+  <!--xacro:include filename="$(find boxbot_description)/xacro/materials.gazebo"/>
   <xacro:gazebo_widowx six_dof="true" head="true"/-->
 </robot>

File: boxbot_description/xacro/head.urdf.xacro (robot description, xacro)
@@ -66,5 +66,5 @@
     <link name="left_camera_link">
       <visual>
-        <origin rpy="0 0 0" xyz="0 0 0"/>
+        <origin rpy="0 ${radians(-90)} 0" xyz="0 0 0"/>
         <geometry>
           <cylinder radius="0.014" length="0.003"/>
@@ -73,5 +73,5 @@
       </visual>
       <collision>
-        <origin rpy="0 0 0" xyz="0 0 0"/>
+        <origin rpy="0 ${radians(-90)} 0" xyz="0 0 0"/>
         <geometry>
           <cylinder radius="0.014" length="0.003"/>
@@ -79,5 +79,5 @@
       </collision>
       <inertial>
-        <origin xyz="0.0 0.0 0.0" rpy="0 0 0" />
+        <origin xyz="0.0 0.0 0.0" rpy="0 ${radians(-90)} 0" />
         <mass value="0.001" />
         <inertia ixx="0.001" ixy="0.0" ixz="0.0" iyy="0.001" iyz="0.0" izz="0.001" />
@@ -86,5 +86,5 @@
     <link name="right_camera_link">
       <visual>
-        <origin rpy="0 0 0" xyz="0 0 0"/>
+        <origin rpy="0 ${radians(-90)} 0" xyz="0 0 0"/>
         <geometry>
           <cylinder radius="0.014" length="0.003"/>
@@ -93,5 +93,5 @@
       </visual>
       <collision>
-        <origin rpy="0 0 0" xyz="0 0 0"/>
+        <origin rpy="0 ${radians(-90)} 0" xyz="0 0 0"/>
         <geometry>
           <cylinder radius="0.014" length="0.003"/>
@@ -99,5 +99,5 @@
       </collision>
       <inertial>
-        <origin xyz="0.0 0.0 0.0" rpy="0 0 0" />
+        <origin xyz="0.0 0.0 0.0" rpy="0 ${radians(-90)} 0" />
         <mass value="0.001" />
         <inertia ixx="0.001" ixy="0.0" ixz="0.0" iyy="0.001" iyz="0.0" izz="0.001" />
@@ -125,21 +125,16 @@
     </joint>
     <joint name="left_camera_joint" type="fixed">
-      <origin rpy="0 ${radians(-90)} 0" xyz="0.023 0.045 0.005"/>
+      <origin rpy="0 0 0" xyz="0.023 0.045 0.005"/>
       <parent link="tilt_link" />
       <child link="left_camera_link"/>
     </joint>
     <joint name="right_camera_joint" type="fixed">
-      <origin rpy="0 ${radians(-90)} 0" xyz="0.023 -0.045 0.005"/>
+      <origin rpy="0 0 0" xyz="0.023 -0.045 0.005"/>
       <parent link="tilt_link" />
       <child link="right_camera_link"/>
     </joint>
-    <!--xacro:include filename="$(find boxbot_description)/xacro/camera.xacro"/>
-    <xacro:rgb_camera parent="tilt_link" prefix="left_">
-      <origin rpy="0 ${radians(-90)} 0" xyz="0.023 0.045 0.005"/>
-    </xacro:rgb_camera>
     <xacro:include filename="$(find boxbot_description)/xacro/camera.xacro"/>
-    <xacro:rgb_camera parent="tilt_link" prefix="right_">
-      <origin rpy="0 ${radians(-90)} 0" xyz="0.023 -0.045 0.005"/>
-    </xacro:rgb_camera-->
+    <xacro:rgb_camera prefix="left_"/>
+    <xacro:rgb_camera prefix="right_"/>
   </xacro:macro>
 </robot>

Commit message: Update URDF model appearance

File: boxbot_description/robots/boxbot_5dof.urdf.xacro (robot description, xacro)
@@ -10,5 +10,5 @@
         <mesh filename="package://boxbot_description/meshes/torso_link.stl"/>
       </geometry>
-      <xacro:material_yellow/>
+      <xacro:material_ivory/>
     </visual>
     <collision>
@@ -52,5 +52,3 @@
     </plugin>
   </gazebo>
-  <!--xacro:include filename="$(find boxbot_description)/xacro/materials.gazebo"/>
-  <xacro:gazebo_widowx six_dof="true" head="true"/-->
 </robot>

File: boxbot_description/robots/boxbot_6dof.urdf.xacro (robot description, xacro)
@@ -10,5 +10,5 @@
         <mesh filename="package://boxbot_description/meshes/torso_link.stl"/>
       </geometry>
-      <xacro:material_yellow/>
+      <xacro:material_ivory/>
     </visual>
     <collision>
@@ -52,5 +52,3 @@
     </plugin>
   </gazebo>
-  <!--xacro:include filename="$(find boxbot_description)/xacro/materials.gazebo"/>
-  <xacro:gazebo_widowx six_dof="true" head="true"/-->
 </robot>

File: boxbot_description/xacro/common_colours.xacro (robot description, xacro)
@@ -8,5 +8,6 @@
 	<xacro:property name="color_grey"     value="0.34 0.35 0.36 1.0" />
 	<!-- approximations -->
-	<xacro:property name="color_black"    value="0.15 0.15 0.15 1.0" />
+	<xacro:property name="color_black"    value="0.05 0.05 0.05 1.0" />
 	<xacro:property name="color_greyish"  value="0.75 0.75 0.75 1.0" />
+	<xacro:property name="color_ivory"   value="0.86 0.76 0.35 1.0" />
 </robot>

File: boxbot_description/xacro/common_materials.xacro (robot description, xacro)
@@ -27,3 +27,8 @@
 		</material>
 	</xacro:macro>
+	<xacro:macro name="material_ivory">
+		<material name="">
+			<color rgba="${color_ivory}"/>
+		</material>
+	</xacro:macro>
 </robot>

Commit message: Remove unrequired elements for new version

File: boxbot_description/robots/boxbot_5dof.urdf.xacro (robot description, xacro)
@@ -52,3 +52,5 @@
     </plugin>
   </gazebo>
+  <xacro:include filename="$(find boxbot_description)/xacro/gazebo_materials.xacro"/>
+  <xacro:gazebo_boxbot six_dof="false" head="true"/>
 </robot>

File: boxbot_description/robots/boxbot_6dof.urdf.xacro (robot description, xacro)
@@ -52,3 +52,5 @@
     </plugin>
   </gazebo>
+  <xacro:include filename="$(find boxbot_description)/xacro/gazebo_materials.xacro"/>
+  <xacro:gazebo_boxbot six_dof="true" head="true"/>
 </robot>

File: boxbot_description/xacro/gazebo_materials.xacro (robot description, xacro)
@@ -1,10 +1,9 @@
 <?xml version="1.0"?>
 <robot xmlns:xacro="http://ros.org/wiki/xacro">
-  <xacro:macro name="gazebo_widowx" params="six_dof head">
+  <xacro:macro name="gazebo_boxbot" params="six_dof head">
   <!--Gazebo compatable colors-->
     <gazebo reference="torso">
       <mu1>0.3</mu1>
       <mu2>0.3</mu2>
-      <material>Gazebo/Wood</material>
     </gazebo>
     <!--left arm-->
@@ -12,15 +11,12 @@
       <mu1>0.6</mu1>
       <mu2>0.6</mu2>
-      <material>Gazebo/DarkGrey</material>
     </gazebo>
     <gazebo reference="left_biceps_link">
       <mu1>0.6</mu1>
       <mu2>0.6</mu2>
-      <material>Gazebo/DarkGrey</material>
     </gazebo>
     <gazebo reference="left_forearm_1_link">
       <mu1>0.6</mu1>
       <mu2>0.6</mu2>
-      <material>Gazebo/DarkGrey</material>
     </gazebo>
     <xacro:if value="${six_dof}">
@@ -28,5 +24,4 @@
         <mu1>0.6</mu1>
         <mu2>0.6</mu2>
-        <material>Gazebo/DarkGrey</material>
       </gazebo>
     </xacro:if>
@@ -34,25 +29,20 @@
       <mu1>0.6</mu1>
       <mu2>0.6</mu2>
-      <material>Gazebo/DarkGrey</material>
     </gazebo>
     <gazebo reference="left_wrist_2_link">
       <mu1>0.6</mu1>
       <mu2>0.6</mu2>
-      <material>Gazebo/DarkGrey</material>
     </gazebo>
     <gazebo reference="left_gripper_rail_link">
       <mu1>0.6</mu1>
       <mu2>0.6</mu2>
-      <material>Gazebo/DarkGrey</material>
     </gazebo>
     <gazebo reference="left_gripper_1_link">
       <mu1>1.0</mu1>
       <mu2>1.0</mu2>
-      <material>Gazebo/DarkGrey</material>
     </gazebo>
     <gazebo reference="left_gripper_2_link">
       <mu1>1.0</mu1>
       <mu2>1.0</mu2>
-      <material>Gazebo/DarkGrey</material>
     </gazebo>
     <!--right arm-->
@@ -60,15 +50,12 @@
       <mu1>0.6</mu1>
       <mu2>0.6</mu2>
-      <material>Gazebo/DarkGrey</material>
     </gazebo>
     <gazebo reference="right_biceps_link">
       <mu1>0.6</mu1>
       <mu2>0.6</mu2>
-      <material>Gazebo/DarkGrey</material>
     </gazebo>
     <gazebo reference="right_forearm_1_link">
       <mu1>0.6</mu1>
       <mu2>0.6</mu2>
-      <material>Gazebo/DarkGrey</material>
     </gazebo>
     <xacro:if value="${six_dof}">
@@ -76,5 +63,4 @@
         <mu1>0.6</mu1>
         <mu2>0.6</mu2>
-        <material>Gazebo/DarkGrey</material>
       </gazebo>
     </xacro:if>
@@ -82,25 +68,20 @@
       <mu1>0.6</mu1>
       <mu2>0.6</mu2>
-      <material>Gazebo/DarkGrey</material>
     </gazebo>
     <gazebo reference="right_wrist_2_link">
       <mu1>0.6</mu1>
       <mu2>0.6</mu2>
-      <material>Gazebo/DarkGrey</material>
     </gazebo>
     <gazebo reference="right_gripper_rail_link">
       <mu1>0.6</mu1>
       <mu2>0.6</mu2>
-      <material>Gazebo/DarkGrey</material>
     </gazebo>
     <gazebo reference="right_gripper_1_link">
       <mu1>1.0</mu1>
       <mu2>1.0</mu2>
-      <material>Gazebo/DarkGrey</material>
     </gazebo>
     <gazebo reference="right_gripper_2_link">
       <mu1>1.0</mu1>
       <mu2>1.0</mu2>
-      <material>Gazebo/DarkGrey</material>
     </gazebo>
      <xacro:if value="${head}">
@@ -108,5 +89,4 @@
         <mu1>0.6</mu1>
         <mu2>0.6</mu2>
-        <material>Gazebo/DarkGrey</material>
       </gazebo>
     </xacro:if>
@@ -115,5 +95,4 @@
         <mu1>0.6</mu1>
         <mu2>0.6</mu2>
-        <material>Gazebo/DarkGrey</material>
       </gazebo>
     </xacro:if>
@@ -122,5 +101,4 @@
         <mu1>0.6</mu1>
         <mu2>0.6</mu2>
-        <material>Gazebo/DarkGrey</material>
       </gazebo>
     </xacro:if>
@@ -129,5 +107,4 @@
         <mu1>0.6</mu1>
         <mu2>0.6</mu2>
-        <material>Gazebo/DarkGrey</material>
       </gazebo>
     </xacro:if>
@@ -136,5 +113,4 @@
         <mu1>0.6</mu1>
         <mu2>0.6</mu2>
-        <material>Gazebo/DarkGrey</material>
       </gazebo>
     </xacro:if>
