Commit message: Add some new scenarios.

File: boxbot_gazebo/models/block_1.urdf.xacro (robot description, xacro)
@@ -4,5 +4,5 @@
     <inertial>
       <origin xyz="0.0 0.0 0.0"/>
-      <mass value="0.14"/>
+      <mass value="0.05"/>
       <inertia ixx="0.001" ixy="0.0" ixz="0.0" iyy="0.001" iyz="0.0" izz="0.001"/>
     </inertial>
@@ -21,4 +21,6 @@
   </link>
   <gazebo reference="link_1">
+    <mu1>500.0</mu1>
+    <mu2>500.0</mu2>
     <material>Gazebo/Wood</material>
   </gazebo>

Commit message: Add contact sensor to block_1; add more scenarios.

File: boxbot_gazebo/models/block_1.urdf.xacro (robot description, xacro)
@@ -24,4 +24,15 @@
     <mu2>1.0</mu2>
     <material>Gazebo/Wood</material>
+    <sensor name="block_contact" type="contact">
+      <always_on>true</always_on>
+      <update_rate>30</update_rate>
+      <contact>
+        <collision>link_1_collision</collision>
+      </contact>
+      <plugin name="block_contact_plugin" filename="libgazebo_ros_bumper.so">
+        <bumperTopicName>block_contact_state</bumperTopicName>
+        <frameName>link_1</frameName>
+      </plugin>
+    </sensor>
   </gazebo>
 </robot>
