Commit message: Fix some incorrect paths for the workspace models

File: boxbot_workspace/urdf/eva_cable.urdf.xacro (robot description, xacro)
@@ -67,5 +67,5 @@
     <material>Gazebo/FlatBlack</material>
   </gazebo>
-  <xacro:include filename="$(find bb_workspace)/urdf/cable.xacro"/>
+  <xacro:include filename="$(find boxbot_workspace)/urdf/cable.xacro"/>
   <xacro:cable_segment number="1" parent="0" radius="${radius}" length="${length}" effort="${effort}" velocity="${velocity}" damping="${damping}" friction="${friction}"/>
   <xacro:cable_segment number="2" parent="1" radius="${radius}" length="${length}" effort="${effort}" velocity="${velocity}" damping="${damping}" friction="${friction}"/>
@@ -91,5 +91,5 @@
       <origin rpy="0.0 0.0 0.0" xyz="0.0 0.0 ${length/2}"/>
       <geometry>
-        <mesh filename="package://bb_workspace/meshes/plug.stl" scale="0.001 0.001 0.001"/>
+        <mesh filename="package://boxbot_workspace/meshes/plug.stl" scale="0.001 0.001 0.001"/>
       </geometry>
     </visual>
@@ -97,5 +97,5 @@
       <origin rpy="0.0 0.0 0.0" xyz="0.0 0.0 ${length/2}"/>
       <geometry>
-        <mesh filename="package://bb_workspace/meshes/plug.stl" scale="0.001 0.001 0.001"/>
+        <mesh filename="package://boxbot_workspace/meshes/plug.stl" scale="0.001 0.001 0.001"/>
       </geometry>
     </collision>
